File: i3c.kicad_sch (KiCad schematic)
At the start: 4 parts, among them U25 MMC5603NJ

Commit message: *.kicad_sch: ERC clean
Signed-off-by: Huang Rui <vowstar@gmail.com>
Connections:
- net P12V renamed VDD
Changed lines of the file:
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@@
   )
   (bus_alias "I3C" (members "SCL" "SDA"))
+  (junction (at 143.51 62.23) (diameter 0) (color 0 0 0 0)
+  )
+  (junction (at 147.32 82.55) (diameter 0) (color 0 0 0 0)
+  )
   (junction (at 95.25 74.93) (diameter 0) (color 0 0 0 0)
   )
-  (junction (at 147.32 82.55) (diameter 0) (color 0 0 0 0)
-  )
-  (junction (at 143.51 62.23) (diameter 0) (color 0 0 0 0)
-  )
   (junction (at 95.25 82.55) (diameter 0) (color 0 0 0 0)
   )
@@
     (stroke (width 0) (type default))
   )
+  (bus (pts (xy 160.02 72.39) (xy 160.02 80.01))
+    (stroke (width 0) (type default))
+  )
+  (wire (pts (xy 95.25 74.93) (xy 106.68 74.93))
+    (stroke (width 0) (type default))
+  )
   (wire (pts (xy 143.51 62.23) (xy 147.32 62.23))
     (stroke (width 0) (type default))
   )
+  (wire (pts (xy 147.32 63.5) (xy 147.32 62.23))
+    (stroke (width 0) (type default))
+  )
   (wire (pts (xy 139.7 62.23) (xy 143.51 62.23))
-    (stroke (width 0) (type default))
-  )
-  (bus (pts (xy 160.02 72.39) (xy 160.02 80.01))
-    (stroke (width 0) (type default))
-  )
-  (wire (pts (xy 95.25 74.93) (xy 106.68 74.93))
-    (stroke (width 0) (type default))
-  )
-  (wire (pts (xy 147.32 63.5) (xy 147.32 62.23))
     (stroke (width 0) (type default))
   )
@@
     (effects (font (size 1.27 1.27)) (justify left))
   )
+  (symbol (lib_id "Device:R") (at 147.32 67.31 0) (unit 1)
+    (in_bom yes) (on_board yes) (dnp no) (fields_autoplaced)
+    (property "Reference" "R43" (at 149.86 66.675 0)
+      (effects (font (size 1.27 1.27)) (justify left))
+    )
+    (property "Value" "10k" (at 149.86 69.215 0)
+      (effects (font (size 1.27 1.27)) (justify left))
+    )
+    (property "Footprint" "Resistor_SMD:R_0402_1005Metric" (at 145.542 67.31 90)
+      (effects (font (size 1.27 1.27)) hide)
+    )
+    (property "Datasheet" "~" (at 147.32 67.31 0)
+      (effects (font (size 1.27 1.27)) hide)
+    )
+    (pin "1")
+    (pin "2")
+    (instances
+      (project "fmc_usb_gpio_spi_jtag"
+        (path "/387bfcf1-ae49-4b85-be89-3bb02ce2e960/2664394d-fb06-44a8-a976-124c25ea0771"
+          (reference "R43") (unit 1)
+        )
+      )
+      (project "compass_board"
+        (path "/e4400406-c137-4d46-a41d-a5d0f4ed8ce2"
+          (reference "R2") (unit 1)
+        )
+      )
+    )
+  )
   (symbol (lib_id "power:VDD") (at 95.25 74.93 0) (unit 1)
-    (in_bom yes) (on_board yes) (dnp no)
-    (property "Reference" "#PWR01" (at 95.25 78.74 0)
-      (effects (font (size 1.27 1.27)) hide)
-    )
-    (property "Value" "VADJ" (at 92.71 71.12 0)
+    (in_bom yes) (on_board yes) (dnp no) (fields_autoplaced)
+    (property "Reference" "#PWR096" (at 95.25 78.74 0)
+      (effects (font (size 1.27 1.27)) hide)
+    )
+    (property "Value" "VADJ" (at 95.25 71.12 0)
       (effects (font (size 1.27 1.27)))
     )
@@
     (instances
       (project "fmc_usb_gpio_spi_jtag"
-        (path "/387bfcf1-ae49-4b85-be89-3bb02ce2e960/4338fda8-0ea2-4bf2-b1c2-c685ef11d6a0"
-          (reference "#PWR01") (unit 1)
-        )
-        (path "/387bfcf1-ae49-4b85-be89-3bb02ce2e960/4ff80468-3372-4da6-9aa6-0708696df1f4"
-          (reference "#PWR083") (unit 1)
-        )
-        (path "/387bfcf1-ae49-4b85-be89-3bb02ce2e960/dc9f6e10-2e8e-48ac-b16a-cc17c057f50a"
-          (reference "#PWR087") (unit 1)
-        )
-        (path "/387bfcf1-ae49-4b85-be89-3bb02ce2e960/050a965f-1566-4fd5-8eeb-6ab96a9baeba"
-          (reference "#PWR0113") (unit 1)
-        )
-        (path "/387bfcf1-ae49-4b85-be89-3bb02ce2e960/9cd800a1-5b4a-4dab-b708-f8f78f4f7813"
-          (reference "#PWR0238") (unit 1)
-        )
-        (path "/387bfcf1-ae49-4b85-be89-3bb02ce2e960/2664394d-fb06-44a8-a976-124c25ea0771"
-          (reference "#PWR0266") (unit 1)
-        )
-      )
-    )
-  )
-  (symbol (lib_id "Device:R") (at 147.32 67.31 0) (unit 1)
-    (in_bom yes) (on_board yes) (dnp no) (fields_autoplaced)
-    (property "Reference" "R43" (at 149.86 66.675 0)
-      (effects (font (size 1.27 1.27)) (justify left))
-    )
-    (property "Value" "10k" (at 149.86 69.215 0)
-      (effects (font (size 1.27 1.27)) (justify left))
-    )
-    (property "Footprint" "Resistor_SMD:R_0402_1005Metric" (at 145.542 67.31 90)
-      (effects (font (size 1.27 1.27)) hide)
-    )
-    (property "Datasheet" "~" (at 147.32 67.31 0)
-      (effects (font (size 1.27 1.27)) hide)
-    )
-    (pin "1")
-    (pin "2")
-    (instances
-      (project "fmc_usb_gpio_spi_jtag"
-        (path "/387bfcf1-ae49-4b85-be89-3bb02ce2e960/2664394d-fb06-44a8-a976-124c25ea0771"
-          (reference "R43") (unit 1)
-        )
-      )
-      (project "compass_board"
-        (path "/e4400406-c137-4d46-a41d-a5d0f4ed8ce2"
-          (reference "R2") (unit 1)
+        (path "/387bfcf1-ae49-4b85-be89-3bb02ce2e960/2664394d-fb06-44a8-a976-124c25ea0771"
+          (reference "#PWR096") (unit 1)
+        )
+      )
+    )
+  )
+  (symbol (lib_id "power:VDD") (at 143.51 62.23 0) (unit 1)
+    (in_bom yes) (on_board yes) (dnp no) (fields_autoplaced)
+    (property "Reference" "#PWR098" (at 143.51 66.04 0)
+      (effects (font (size 1.27 1.27)) hide)
+    )
+    (property "Value" "VADJ" (at 143.51 58.42 0)
+      (effects (font (size 1.27 1.27)))
+    )
+    (property "Footprint" "" (at 143.51 62.23 0)
+      (effects (font (size 1.27 1.27)) hide)
+    )
+    (property "Datasheet" "" (at 143.51 62.23 0)
+      (effects (font (size 1.27 1.27)) hide)
+    )
+    (pin "1")
+    (instances
+      (project "fmc_usb_gpio_spi_jtag"
+        (path "/387bfcf1-ae49-4b85-be89-3bb02ce2e960/2664394d-fb06-44a8-a976-124c25ea0771"
+          (reference "#PWR098") (unit 1)
         )
       )
@@
         )
       )
-    )
-  )
-  (symbol (lib_id "power:VDD") (at 143.51 62.23 0) (unit 1)
-    (in_bom yes) (on_board yes) (dnp no)
-    (property "Reference" "#PWR01" (at 143.51 66.04 0)
-      (effects (font (size 1.27 1.27)) hide)
-    )
-    (property "Value" "VADJ" (at 140.97 58.42 0)
-      (effects (font (size 1.27 1.27)))
-    )
-    (property "Footprint" "" (at 143.51 62.23 0)
-      (effects (font (size 1.27 1.27)) hide)
-    )
-    (property "Datasheet" "" (at 143.51 62.23 0)
-      (effects (font (size 1.27 1.27)) hide)
-    )
-    (pin "1")
-    (instances
-      (project "fmc_usb_gpio_spi_jtag"
-        (path "/387bfcf1-ae49-4b85-be89-3bb02ce2e960/4338fda8-0ea2-4bf2-b1c2-c685ef11d6a0"
-          (reference "#PWR01") (unit 1)
-        )
-        (path "/387bfcf1-ae49-4b85-be89-3bb02ce2e960/4ff80468-3372-4da6-9aa6-0708696df1f4"
-          (reference "#PWR083") (unit 1)
-        )
-        (path "/387bfcf1-ae49-4b85-be89-3bb02ce2e960/dc9f6e10-2e8e-48ac-b16a-cc17c057f50a"
-          (reference "#PWR087") (unit 1)
-        )
-        (path "/387bfcf1-ae49-4b85-be89-3bb02ce2e960/050a965f-1566-4fd5-8eeb-6ab96a9baeba"
-          (reference "#PWR0113") (unit 1)
-        )
-        (path "/387bfcf1-ae49-4b85-be89-3bb02ce2e960/9cd800a1-5b4a-4dab-b708-f8f78f4f7813"
-          (reference "#PWR0238") (unit 1)
-        )
-        (path "/387bfcf1-ae49-4b85-be89-3bb02ce2e960/2664394d-fb06-44a8-a976-124c25ea0771"
-          (reference "#PWR0264") (unit 1)
-        )
-      )

Commit message: {library,*.kicad_sch}: fix power symbols, ERC clean
Signed-off-by: Huang Rui <vowstar@gmail.com>
Connections:
- net VDD renamed VADJ
Changed lines of the file:
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@@
     )
   )
-  (symbol (lib_id "power:VDD") (at 95.25 74.93 0) (unit 1)
+  (symbol (lib_id "CHIPSAlliance_Power:VADJ") (at 95.25 74.93 0) (unit 1)
     (in_bom yes) (on_board yes) (dnp no) (fields_autoplaced)
     (property "Reference" "#PWR096" (at 95.25 78.74 0)
@@
     )
   )
-  (symbol (lib_id "power:VDD") (at 143.51 62.23 0) (unit 1)
+  (symbol (lib_id "CHIPSAlliance_Power:VADJ") (at 143.51 62.23 0) (unit 1)
     (in_bom yes) (on_board yes) (dnp no) (fields_autoplaced)
     (property "Reference" "#PWR098" (at 143.51 66.04 0)
@@
     )
   )
-  (symbol (lib_id "power:GND") (at 95.25 82.55 0) (unit 1)
+  (symbol (lib_id "CHIPSAlliance_Power:GND") (at 95.25 82.55 0) (unit 1)
     (in_bom yes) (on_board yes) (dnp no) (fields_autoplaced)
     (property "Reference" "#PWR0265" (at 95.25 88.9 0)
