File: power.kicad_sch (KiCad schematic)
At the start: 21 parts, among them U13 MT2492, U4 AIP74LVC1T45GB236TR

Commit message: *.kicad_sch: apply new template styles
Signed-off-by: Huang Rui <vowstar@gmail.com>
Other:
- company: (none) -> CHIPS Alliance
- title: (none) -> POWER
Changed lines of the file:
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@@
 (kicad_sch (version 20230121) (generator eeschema)
   (paper "A4")
+  (title_block
+    (title "POWER")
+    (date "2023-03-02")
+    (rev "1.0.0")
+    (company "CHIPS Alliance")
+    (comment 1 "Rui Huang (2023-03-02)")
+    (comment 2 "Rui Huang (2023-03-02)")
+    (comment 4 "Rui Huang (2023-03-02)")
+  )
   (junction (at 62.23 74.93) (diameter 0) (color 0 0 0 0)
   )

Commit message: *.kicad_sch: ERC clean
Signed-off-by: Huang Rui <vowstar@gmail.com>
Parts:
- added R1 (x3): 10k, Resistor_SMD:R_0402_1005Metric, symbol Device:R
Connections:
- net GND: now also U13.2 (GND); no longer U13.1 (GND)
- net VDD: now also C24.1, D12.1 (VDD), U13.4 (EN), U13.5 (IN), U4.1 (VCCA), U4.1 (VCCA), U4.1 (VCCA), U4.1 (VCCA), U4.6 (VCCB), U4.6 (VCCB), U4.6 (VCCB), U4.6 (VCCB), R1.1, R1.1, R1.1
- net at C1.1, R1.1, R1.2: now also U13.3 (FB); no longer U13.4 (FB)
- net at C1.1, L1.1: now also U13.6 (SW); no longer U13.2 (SW)
- net at C1.2: now also U13.1 (BST); no longer U13.6 (BST)
- removed net P12V: C24.1, D12.1 (VDD), U13.3 (IN), U13.5 (EN), U4.1 (VCCA), U4.1 (VCCA), U4.1 (VCCA), U4.1 (VCCA), U4.4 (B), U4.4 (B), U4.4 (B), U4.6 (VCCB), U4.6 (VCCB), U4.6 (VCCB), U4.6 (VCCB)
- new net: R1.2, U4.4 (B) (x3)

Commit message: {library,*.kicad_sch}: fix power symbols, ERC clean
Signed-off-by: Huang Rui <vowstar@gmail.com>
Connections:
- net VDD renamed 5P0V
- net 5P0V: no longer C24.1, R1.1, R1.1, R1.1, U13.4 (EN), U13.5 (IN), U4.6 (VCCB), U4.6 (VCCB), U4.6 (VCCB), U4.6 (VCCB)
- new net 12P0V: C24.1, U13.4 (EN), U13.5 (IN)
- new net 3P3V: R1.1, U4.6 (VCCB)
- new net 3P3VAUX: R1.1, U4.6 (VCCB)
- new net VADJ: R1.1, U4.6 (VCCB), U4.6 (VCCB)
