File: uart.kicad_sch (KiCad schematic)
At the start: 28 parts, among them J3 USB_C_Receptacle, U12 TPD4E02B04DQA, U14 TXS02612RTWR, U3 CP2104

Commit message: *.*: fix USB_C_Receptacle_Molex_105450-0101 3d model
Signed-off-by: Huang Rui <vowstar@gmail.com>
Parts:
- J3: footprint Connector_USB:USB_C_Receptacle_Molex_105450-0101 -> CHIPSAlliance_Connector:USB_C_Receptacle_Molex_105450-0101
Changed lines of the file:
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@@
     (comment 4 "Rui Huang (2023-03-02)")
   )
+  (bus_alias "SDIO" (members "DAT0" "DAT1" "DAT2" "DAT3" "CMD" "CLK"))
   (bus_alias "UART" (members "TXD" "RXD" "~{RTS}" "~{CTS}" "~{DSR}" "~{DTR}" "~{DCD}" "~{RI}"))
-  (bus_alias "SDIO" (members "DAT0" "DAT1" "DAT2" "DAT3" "CMD" "CLK"))
   (junction (at 182.88 60.96) (diameter 0) (color 0 0 0 0)
   )
@@
   (junction (at 187.96 60.96) (diameter 0) (color 0 0 0 0)
   )
+  (junction (at 180.34 60.96) (diameter 0) (color 0 0 0 0)
+  )
+  (junction (at 245.11 93.98) (diameter 0) (color 0 0 0 0)
+  )
+  (junction (at 125.73 96.52) (diameter 0) (color 0 0 0 0)
+  )
+  (junction (at 212.09 100.33) (diameter 0) (color 0 0 0 0)
+  )
+  (junction (at 48.26 125.73) (diameter 0) (color 0 0 0 0)
+  )
+  (junction (at 212.09 96.52) (diameter 0) (color 0 0 0 0)
+  )
+  (junction (at 223.52 86.36) (diameter 0) (color 0 0 0 0)
+  )
+  (junction (at 217.17 100.33) (diameter 0) (color 0 0 0 0)
+  )
   (junction (at 245.11 96.52) (diameter 0) (color 0 0 0 0)
   )
-  (junction (at 180.34 60.96) (diameter 0) (color 0 0 0 0)
-  )
-  (junction (at 125.73 96.52) (diameter 0) (color 0 0 0 0)
-  )
-  (junction (at 212.09 100.33) (diameter 0) (color 0 0 0 0)
-  )
-  (junction (at 48.26 125.73) (diameter 0) (color 0 0 0 0)
-  )
-  (junction (at 212.09 96.52) (diameter 0) (color 0 0 0 0)
-  )
-  (junction (at 223.52 86.36) (diameter 0) (color 0 0 0 0)
-  )
-  (junction (at 217.17 100.33) (diameter 0) (color 0 0 0 0)
-  )
   (junction (at 125.73 91.44) (diameter 0) (color 0 0 0 0)
-  )
-  (junction (at 245.11 93.98) (diameter 0) (color 0 0 0 0)
   )
   (junction (at 217.17 93.98) (diameter 0) (color 0 0 0 0)
@@
     )
   )
+  (symbol (lib_id "CHIPSAlliance_Power:GND") (at 172.72 68.58 0) (unit 1)
+    (in_bom yes) (on_board yes) (dnp no)
+    (property "Reference" "#PWR02" (at 172.72 74.93 0)
+      (effects (font (size 1.27 1.27)) hide)
+    )
+    (property "Value" "GND" (at 172.72 72.39 0)
+      (effects (font (size 1.27 1.27)))
+    )
+    (property "Footprint" "" (at 172.72 68.58 0)
+      (effects (font (size 1.27 1.27)) hide)
+    )
+    (property "Datasheet" "" (at 172.72 68.58 0)
+      (effects (font (size 1.27 1.27)) hide)
+    )
+    (pin "1")
+    (instances
+      (project "fmc_usb_gpio_spi_jtag"
+        (path "/387bfcf1-ae49-4b85-be89-3bb02ce2e960/4338fda8-0ea2-4bf2-b1c2-c685ef11d6a0"
+          (reference "#PWR02") (unit 1)
+        )
+        (path "/387bfcf1-ae49-4b85-be89-3bb02ce2e960/4ff80468-3372-4da6-9aa6-0708696df1f4"
+          (reference "#PWR099") (unit 1)
+        )
+        (path "/387bfcf1-ae49-4b85-be89-3bb02ce2e960/050a965f-1566-4fd5-8eeb-6ab96a9baeba"
+          (reference "#PWR0102") (unit 1)
+        )
+      )
+    )
+  )
+  (symbol (lib_id "Device:R") (at 115.57 96.52 90) (unit 1)
+    (in_bom yes) (on_board yes) (dnp no)
+    (property "Reference" "R1" (at 110.49 95.25 90)
+      (effects (font (size 1.27 1.27)))
+    )
+    (property "Value" "10k" (at 120.65 95.25 90)
+      (effects (font (size 1.27 1.27)))
+    )
+    (property "Footprint" "Resistor_SMD:R_0402_1005Metric" (at 115.57 98.298 90)
+      (effects (font (size 1.27 1.27)) hide)
+    )
+    (property "Datasheet" "~" (at 115.57 96.52 0)
+      (effects (font (size 1.27 1.27)) hide)
+    )
+    (pin "1")
+    (pin "2")
+    (instances
+      (project "fmc_usb_gpio_spi_jtag"
+        (path "/387bfcf1-ae49-4b85-be89-3bb02ce2e960/4ff80468-3372-4da6-9aa6-0708696df1f4"
+          (reference "R1") (unit 1)
+        )
+        (path "/387bfcf1-ae49-4b85-be89-3bb02ce2e960/050a965f-1566-4fd5-8eeb-6ab96a9baeba"
+          (reference "R9") (unit 1)
+        )
+      )
+    )
+  )
+  (symbol (lib_id "CHIPSAlliance_Power:GND") (at 74.93 125.73 0) (unit 1)
+    (in_bom yes) (on_board yes) (dnp no) (fields_autoplaced)
+    (property "Reference" "#PWR0266" (at 74.93 132.08 0)
+      (effects (font (size 1.27 1.27)) hide)
+    )
+    (property "Value" "GND" (at 74.93 130.81 0)
+      (effects (font (size 1.27 1.27)))
+    )
+    (property "Footprint" "" (at 74.93 125.73 0)
+      (effects (font (size 1.27 1.27)) hide)
+    )
+    (property "Datasheet" "" (at 74.93 125.73 0)
+      (effects (font (size 1.27 1.27)) hide)
+    )
+    (pin "1")
+    (instances
+      (project "fmc_usb_gpio_spi_jtag"
+        (path "/387bfcf1-ae49-4b85-be89-3bb02ce2e960/8f11314c-d9eb-415d-8d76-07f3be42979a"
+          (reference "#PWR0266") (unit 1)
+        )
+        (path "/387bfcf1-ae49-4b85-be89-3bb02ce2e960/050a965f-1566-4fd5-8eeb-6ab96a9baeba"
+          (reference "#PWR0281") (unit 1)
+        )
+      )
+    )
+  )
   (symbol (lib_id "CHIPSAlliance_Connector:USB_C_Receptacle") (at 270.51 76.2 0) (mirror y) (unit 1)
     (in_bom yes) (on_board yes) (dnp no)
@@
       (effects (font (size 1.27 1.27)))
     )
-    (property "Footprint" "Connector_USB:USB_C_Receptacle_Molex_105450-0101" (at 270.51 143.51 0)
+    (property "Footprint" "CHIPSAlliance_Connector:USB_C_Receptacle_Molex_105450-0101" (at 270.51 143.51 0)
       (effects (font (size 1.27 1.27)) (justify left) hide)
     )
@@
         )
       )
-    )
-  )
-  (symbol (lib_id "CHIPSAlliance_Power:GND") (at 172.72 68.58 0) (unit 1)
-    (in_bom yes) (on_board yes) (dnp no)
-    (property "Reference" "#PWR02" (at 172.72 74.93 0)
-      (effects (font (size 1.27 1.27)) hide)
-    )
-    (property "Value" "GND" (at 172.72 72.39 0)
-      (effects (font (size 1.27 1.27)))
-    )
-    (property "Footprint" "" (at 172.72 68.58 0)
-      (effects (font (size 1.27 1.27)) hide)
-    )
-    (property "Datasheet" "" (at 172.72 68.58 0)
-      (effects (font (size 1.27 1.27)) hide)
-    )
-    (pin "1")
-    (instances
-      (project "fmc_usb_gpio_spi_jtag"
-        (path "/387bfcf1-ae49-4b85-be89-3bb02ce2e960/4338fda8-0ea2-4bf2-b1c2-c685ef11d6a0"
-          (reference "#PWR02") (unit 1)
-        )
-        (path "/387bfcf1-ae49-4b85-be89-3bb02ce2e960/4ff80468-3372-4da6-9aa6-0708696df1f4"
-          (reference "#PWR099") (unit 1)
-        )
-        (path "/387bfcf1-ae49-4b85-be89-3bb02ce2e960/050a965f-1566-4fd5-8eeb-6ab96a9baeba"
-          (reference "#PWR0102") (unit 1)
-        )
-      )
-    )
-  )
-  (symbol (lib_id "Device:R") (at 115.57 96.52 90) (unit 1)
-    (in_bom yes) (on_board yes) (dnp no)
-    (property "Reference" "R1" (at 110.49 95.25 90)
-      (effects (font (size 1.27 1.27)))
-    )
-    (property "Value" "10k" (at 120.65 95.25 90)
-      (effects (font (size 1.27 1.27)))
-    )
-    (property "Footprint" "Resistor_SMD:R_0402_1005Metric" (at 115.57 98.298 90)
-      (effects (font (size 1.27 1.27)) hide)
-    )
-    (property "Datasheet" "~" (at 115.57 96.52 0)
-      (effects (font (size 1.27 1.27)) hide)
-    )
-    (pin "1")
-    (pin "2")
-    (instances
-      (project "fmc_usb_gpio_spi_jtag"
-        (path "/387bfcf1-ae49-4b85-be89-3bb02ce2e960/4ff80468-3372-4da6-9aa6-0708696df1f4"
-          (reference "R1") (unit 1)
-        )
-        (path "/387bfcf1-ae49-4b85-be89-3bb02ce2e960/050a965f-1566-4fd5-8eeb-6ab96a9baeba"
-          (reference "R9") (unit 1)
-        )
-      )
-    )
-  )
-  (symbol (lib_id "CHIPSAlliance_Power:GND") (at 74.93 125.73 0) (unit 1)
-    (in_bom yes) (on_board yes) (dnp no) (fields_autoplaced)
-    (property "Reference" "#PWR0266" (at 74.93 132.08 0)
-      (effects (font (size 1.27 1.27)) hide)
-    )
-    (property "Value" "GND" (at 74.93 130.81 0)
-      (effects (font (size 1.27 1.27)))
-    )
-    (property "Footprint" "" (at 74.93 125.73 0)
-      (effects (font (size 1.27 1.27)) hide)
-    )
-    (property "Datasheet" "" (at 74.93 125.73 0)
-      (effects (font (size 1.27 1.27)) hide)
-    )
-    (pin "1")
-    (instances
-      (project "fmc_usb_gpio_spi_jtag"
-        (path "/387bfcf1-ae49-4b85-be89-3bb02ce2e960/8f11314c-d9eb-415d-8d76-07f3be42979a"
-          (reference "#PWR0266") (unit 1)
-        )
-        (path "/387bfcf1-ae49-4b85-be89-3bb02ce2e960/050a965f-1566-4fd5-8eeb-6ab96a9baeba"
-          (reference "#PWR0281") (unit 1)
-        )
-      )
