File: fmc_basic_peripheral/sdio.kicad_sch (KiCad schematic)
At the start: 12 parts, among them J7 Micro_SD_Card_Det2, U14 TXS02612RTWR

Commit message: fmc_basic_peripheral: Migrate to kicad8
- Migrate schematics to kicad8
- Migrate PCB to kicad8
- Clean ERC
- Clean LVS and DRC

Signed-off-by: Huang Rui <vowstar@gmail.com>
Parts:
- renumbered C1 to C39, C1 to C40, D1 to D7, R1 to R12, R1 to R13, R1 to R14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
