File: fmc_basic_peripheral/sdio.kicad_sch (KiCad schematic)
At the start: 12 parts, among them J7 Micro_SD_Card_Det2, U14 TXS02612RTWR

Commit message: fmc_basic_peripheral: update library and preserve schematic connections
Signed-off-by: Huang Rui <vowstar@gmail.com>
Other:
- moved on the sheet: U14
Changed lines of the file:
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@@
 	(symbol
 		(lib_id "CHIPSAlliance_Connector:Micro_SD_Card_Det2")
-		(at 203.2 78.74 0)
+		(at 227.33 92.71 0)
 		(unit 1)
 		(exclude_from_sim no)
@@
 	(symbol
 		(lib_id "CHIPSAlliance_Logic:TXS02612RTWR")
-		(at 85.09 71.12 0)
+		(at 97.79 93.98 0)
 		(unit 1)
 		(exclude_from_sim no)
@@
 		)
 	)
+	(wire (pts (xy 97.79 120.65) (xy 97.79 119.38)) (stroke (width 0) (type default)))
 )
