File: fmc_basic_peripheral/fmc_usb_gpio_spi_jtag.kicad_pcb (KiCad board)
At the start: 6 copper layers, 76.5 x 69 mm, 146 parts, among them J1 SAMTEC_ASP-134604-01, J2 ACA-SPI-004-K02, J3 USB_C_Receptacle, J4 USB_C_Receptacle, J5 Conn_JTAG_20, J6 PM2.54-2x6, J7 Micro_SD_Card_Det2, J8 PM2.54-2x6, SW1 DSHP04TSGET, SW10 TL3342F160QG, SW2 TL3342F160QG, SW7 TL3342F160QG, SW8 TL3342F160QG, SW9 TL3342F160QG, U1 M24C02-FMN, U11 TXS02612RTWR, U12 TPD4E02B04DQA, U13 MT2492, U14 TXS02612RTWR, U15 TXS02612RTWR, U16 TXS02612RTWR, U17 TXS02612RTWR, U18 TPD4E02B04DQA, U19 TPD4E02B04DQA, U2 STUSB03EQR, U20 TPD4E02B04DQA, U22 AIP74LVC1T45GB236TR, U25 MMC5603NJ, U26 TXS02612RTWR, U27 TXS02612RTWR, U3 CH9102F, U4 TXS02612RTWR, U5 AIP74LVC1T45GB236TR

Commit message: fmc_basic_peripheral: update library and preserve schematic connections
Signed-off-by: Huang Rui <vowstar@gmail.com>
Parts:
- J2: footprint CHIPSAlliance_Connector:ACA-SPI-004 -> CHIPSAlliance_Connector:SOIC-Socket_LOTES_ACA-SPI-004_2x04_P1.27mm
- U2: footprint CHIPSAlliance_Interface:QFN_B03EQR_STM -> CHIPSAlliance_Interface:ST_STUSB03EQR_QFN-16-1EP_3x3mm_P0.5mm_EP1.8034x1.8034mm
- U25: footprint CHIPSAlliance_Sensor:WLP4_N40P2X2_80X80X52N -> CHIPSAlliance_Sensor:WLCSP-4_0.8x0.8mm_Layout2x2_P0.4mm_Ball0.22mm_Pad0.25mm_NSMD
