File: fmc_basic_peripheral/gpio.kicad_sch (KiCad schematic)
At the start: 43 parts, among them J6 PM2.54-2x6, J8 PM2.54-2x6, SW1 DSHP04TSGET, SW10 TL3342F160QG, SW2 TL3342F160QG, SW8 TL3342F160QG, SW9 TL3342F160QG, U11 TXS02612RTWR, U15 TXS02612RTWR, U16 TXS02612RTWR, U26 TXS02612RTWR, U4 TXS02612RTWR

Commit message: fmc_basic_peripheral: update library and preserve schematic connections
Signed-off-by: Huang Rui <vowstar@gmail.com>
Other:
- moved on the sheet: U11, U15, U16, U26, U4
Changed lines of the file:
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@@
 	(symbol
 		(lib_id "CHIPSAlliance_Connector:Conn_PMOD_12")
-		(at 256.54 49.53 0)
+		(at 257.81 55.88 0)
 		(unit 1)
 		(exclude_from_sim no)
@@
 	(symbol
 		(lib_id "CHIPSAlliance_Logic:TXS02612RTWR")
-		(at 95.25 104.14 0)
+		(at 107.95 127 0)
 		(unit 1)
 		(exclude_from_sim no)
@@
 	(symbol
 		(lib_id "CHIPSAlliance_Logic:TXS02612RTWR")
-		(at 31.75 40.64 0)
+		(at 44.45 63.5 0)
 		(unit 1)
 		(exclude_from_sim no)
@@
 	(symbol
 		(lib_id "CHIPSAlliance_Logic:TXS02612RTWR")
-		(at 93.98 40.64 0)
+		(at 106.68 63.5 0)
 		(unit 1)
 		(exclude_from_sim no)
@@
 	(symbol
 		(lib_id "CHIPSAlliance_Logic:TXS02612RTWR")
-		(at 31.75 104.14 0)
+		(at 44.45 127 0)
 		(unit 1)
 		(exclude_from_sim no)
@@
 	(symbol
 		(lib_id "CHIPSAlliance_Connector:Conn_PMOD_12")
-		(at 256.54 73.66 0)
+		(at 257.81 80.01 0)
 		(unit 1)
 		(exclude_from_sim no)
@@
 	(symbol
 		(lib_id "CHIPSAlliance_Logic:TXS02612RTWR")
-		(at 157.48 40.64 0)
+		(at 170.18 63.5 0)
 		(unit 1)
 		(exclude_from_sim no)
@@
 		)
 	)
+	(wire (pts (xy 107.95 153.67) (xy 107.95 152.4)) (stroke (width 0) (type default)))
+	(wire (pts (xy 44.45 90.17) (xy 44.45 88.9)) (stroke (width 0) (type default)))
+	(wire (pts (xy 106.68 90.17) (xy 106.68 88.9)) (stroke (width 0) (type default)))
+	(wire (pts (xy 44.45 153.67) (xy 44.45 152.4)) (stroke (width 0) (type default)))
+	(wire (pts (xy 170.18 90.17) (xy 170.18 88.9)) (stroke (width 0) (type default)))
 )
