File: fmc_basic_peripheral/jtag.kicad_sch (KiCad schematic)
At the start: 8 parts, among them J5 Conn_JTAG_20, SW7 TL3342F160QG, U17 TXS02612RTWR

Commit message: fmc_basic_peripheral: update library and preserve schematic connections
Signed-off-by: Huang Rui <vowstar@gmail.com>
Other:
- moved on the sheet: U17
Changed lines of the file:
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@@
 	(symbol
 		(lib_id "CHIPSAlliance_Connector:Conn_JTAG_20")
-		(at 93.98 80.01 0)
+		(at 106.68 97.79 0)
 		(unit 1)
 		(exclude_from_sim no)
@@
 	(symbol
 		(lib_id "CHIPSAlliance_Logic:TXS02612RTWR")
-		(at 157.48 78.74 0)
+		(at 170.18 101.6 0)
 		(unit 1)
 		(exclude_from_sim no)
@@
 		)
 	)
+	(wire (pts (xy 170.18 128.27) (xy 170.18 127)) (stroke (width 0) (type default)))
 )
