File: fmc_basic_peripheral/spi_flash.kicad_sch (KiCad schematic)
At the start: 4 parts, among them J2 ACA-SPI-004-K02, U19 TPD4E02B04DQA, U20 TPD4E02B04DQA

Commit message: fmc_basic_peripheral: update library and preserve schematic connections
Signed-off-by: Huang Rui <vowstar@gmail.com>
Parts:
- J2: footprint CHIPSAlliance_Connector:ACA-SPI-004 -> CHIPSAlliance_Connector:SOIC-Socket_LOTES_ACA-SPI-004_2x04_P1.27mm
Changed lines of the file:
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@@
 	(symbol
 		(lib_id "CHIPSAlliance_Connector:ACA-SPI-004-K02")
-		(at 182.88 101.6 0)
+		(at 187.96 106.68 0)
 		(unit 1)
 		(exclude_from_sim no)
@@
 			)
 		)
-		(property "Footprint" "CHIPSAlliance_Connector:ACA-SPI-004"
+		(property "Footprint" "CHIPSAlliance_Connector:SOIC-Socket_LOTES_ACA-SPI-004_2x04_P1.27mm"
 			(at 182.88 119.38 0)
 			(effects
