File: fmc_basic_peripheral/usb.kicad_sch (KiCad schematic)
At the start: 15 parts, among them J3 USB_C_Receptacle, U18 TPD4E02B04DQA, U2 STUSB03EQR, U5 AIP74LVC1T45GB236TR

Commit message: fmc_basic_peripheral: update library and preserve schematic connections
Signed-off-by: Huang Rui <vowstar@gmail.com>
Parts:
- U2: footprint CHIPSAlliance_Interface:QFN_B03EQR_STM -> CHIPSAlliance_Interface:ST_STUSB03EQR_QFN-16-1EP_3x3mm_P0.5mm_EP1.8034x1.8034mm
Changed lines of the file:
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@@
 	(symbol
 		(lib_id "CHIPSAlliance_Interface:STUSB03EQR")
-		(at 76.2 55.88 0)
+		(at 91.44 76.2 0)
 		(unit 1)
 		(exclude_from_sim no)
@@
 			)
 		)
-		(property "Footprint" "CHIPSAlliance_Interface:QFN_B03EQR_STM"
+		(property "Footprint" "CHIPSAlliance_Interface:ST_STUSB03EQR_QFN-16-1EP_3x3mm_P0.5mm_EP1.8034x1.8034mm"
 			(at 76.2 100.33 0)
 			(effects
@@
 	(symbol
 		(lib_id "CHIPSAlliance_Logic:AIP74LVC1T45GB236TR")
-		(at 82.55 139.7 0)
+		(at 74.93 147.32 0)
 		(mirror y)
 		(unit 1)
@@
 	(symbol
 		(lib_id "CHIPSAlliance_Connector:USB_C_Receptacle")
-		(at 204.47 58.42 0)
+		(at 194.31 88.9 0)
 		(mirror y)
 		(unit 1)
