File: fpga_candelabra/fpga_bank_0.kicad_sch (KiCad schematic)
At the start: 1 part, among them U1 XCVU13P-B2104

Commit message: fpga_candelabra: add ddr4 power and sysmon mcu periph, bump library
Signed-off-by: Yichuan Gao <gaoyichuan000@gmail.com>
Parts:
- U1: footprint (none) -> CHIPSAlliance_Package_BGA:Xilinx_FHGB2104_VU13P_PkgLength
Changed lines of the file:
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@@
 			)
 		)
-		(property "Footprint" ""
+		(property "Footprint" "CHIPSAlliance_Package_BGA:Xilinx_FHGB2104_VU13P_PkgLength"
 			(at 134.62 26.67 0)
 			(effects
