File: fpga_candelabra/power_supply_sodimm.kicad_sch (KiCad schematic)
At the start: 0 parts

Commit message: fpga_candelabra: add ddr4 power and sysmon mcu periph, bump library
Signed-off-by: Yichuan Gao <gaoyichuan000@gmail.com>
Parts:
- added C191, C195, C207, C209: 100nF, Capacitor_SMD:C_0402_1005Metric, symbol Device:C_Small
- added C192: 1nF, Capacitor_SMD:C_0402_1005Metric, symbol Device:C_Small
- added C193, C194: 100uF 6.3V, Capacitor_SMD:C_1206_3216Metric, symbol Device:C_Small
- added C196, C197, C208: 22uF 25V, Capacitor_SMD:C_1206_3216Metric, symbol Device:C_Small
- added C198, C203: 1uF, Capacitor_SMD:C_0402_1005Metric, symbol Device:C_Small
- added C199, C200, C201, C202, C205, C206: 4.7uF 10V, Capacitor_SMD:C_0402_1005Metric, symbol Device:C_Small
- added C204: 2.2nF, Capacitor_SMD:C_0402_1005Metric, symbol Device:C_Small
- added L12: MWSA1004S-1R0MT, Inductor_SMD:L_Sunlord_MWSA1004S, symbol Device:L_Iron
- added L13: MWSA0402S-2R2MT, Inductor_SMD:L_Sunlord_MWSA0402S, symbol Device:L_Iron
- added Q1, Q2, Q3: AON7544, CHIPSAlliance_Package_DFN_QFN:AO_DFN3x3A_8L_EP1_P_DFN-10-1EP_3x3mm_P0.65mm_EP1.98x2.45mm, symbol CHIPSAlliance_Transistor_FET:AON7544
- added R75, R78, R79, R80, R81, R83, R84, R85: 10k, Resistor_SMD:R_0402_1005Metric, symbol Device:R_Small
- added R76: 1R, Resistor_SMD:R_0402_1005Metric, symbol Device:R_Small
- added R77: 4.7R, Resistor_SMD:R_0402_1005Metric, symbol Device:R_Small
- added R82: 1k, Resistor_SMD:R_0402_1005Metric, symbol Device:R_Small
- added R86: 4.7k, Resistor_SMD:R_0402_1005Metric, symbol Device:R_Small
- added R94: 100R, Resistor_SMD:R_0402_1005Metric, symbol Device:R_Small
- added R95: 330R, Resistor_SMD:R_0402_1005Metric, symbol Device:R_Small
- added U18: TPS51716, Package_DFN_QFN:WQFN-20-1EP_3x3mm_P0.4mm_EP1.7x1.7mm, symbol CHIPSAlliance_Regulator_Switching:TPS51716
- added U19: TLV62130x, CHIPSAlliance_Package_DFN_QFN:Texas_RGT0016C_VQFN-16-1EP_3x3mm_P0.5mm_EP1.68x1.68mm, symbol CHIPSAlliance_Regulator_Switching:TLV62130x
Connections:
- new net: Q2.4 (G), Q3.4 (G), U18.11 (DRVL)
- new net: C191.2, L12.1, Q1.1 (S), Q1.2 (S), Q1.3 (S), Q2.5 (D), Q3.5 (D), R77.2, U18.13 (SW)
- new net: C204.1, U19.9 (SS/TR)
- new net: Q1.4 (G), U18.14 (DRVH)
- new net: R76.1, U18.15 (VBST)
- new net: R83.2, U18.18 (TRIP)
- new net: R82.2, U18.19 (MODE)
- new net: R79.2, U18.6 (VREF)
- new net: R79.1, R80.2, U18.8 (REFIN)
- new net: C191.1, R76.2
- new net: R80.1, R81.2
- new net: C192.2, R77.1
- new net: L13.1, U19.1 (SW), U19.2 (SW), U19.3 (SW)
- new net: R85.1, R86.1, U19.5 (FB)
- new net +12V: C195.2, C196.1, C197.1, Q1.5 (D)
- new net +3.3VAUX: R78.1, R84.1, R94.2
- new net +5V: C198.2, C205.1, C206.1, C207.1, U18.12 (V5IN), U19.10 (AVIN), U19.11 (PVIN), U19.12 (PVIN)
- new net DDR4_EN: R75.2, U18.16 (S5), U18.17 (S3), U19.13 (EN)
- new net DDR4_VDDQ: C193.1, C194.1, C199.1, C200.1, L12.2, U18.2 (VLDOIN), U18.9 (VDDQSNS)
- new net DDR4_VDDQ_PG: R78.2, U18.20 (PGOOD)
- new net DDR4_VDDSPD: R94.1, R95.2
- new net DDR4_VPP: C208.1, C209.1, L13.2, R85.2, U19.14 (VOS)
- new net DDR4_VPP_PG: R84.2, U19.4 (PG)
- new net DDR4_VREF: C203.2, U18.5 (VTTREF)
- new net DDR4_VTT: C201.1, C202.1, U18.1 (VTTSNS), U18.3 (VTT)
- new net Earth: C192.1, C193.2, C194.2, C195.1, C196.2, C197.2, C198.1, C199.2, C200.2, C201.2, C202.2, C203.1, C204.2, C205.2, C206.2, C207.2, C208.2, C209.2, Q2.1 (S), Q2.2 (S), Q2.3 (S), Q3.1 (S), Q3.2 (S), Q3.3 (S), R75.1, R81.1, R82.1, R83.1, R86.2, R95.1, U18.10 (PGND), U18.21 (EPAD), U18.4 (VTTGND), U18.7 (GND), U19.15 (PGND), U19.16 (PGND), U19.17 (EPAD), U19.6 (AGND), U19.7 (FSW), U19.8 (DEF)
Other:
- note added: "12V -> 1.2V 10A VDDQ + VTT + VTTREF Controlled by SYSMON (EN shared with VPP)"
- note added: "3.3V AUX -> 2.5V <1mA VDDSPD"
- note added: "5V Main -> 2.5V 0.5A VPP Controlled by SYSMON (EN shared with VDDQ)"
- note added: "Place next to VLDOIN"
- title: (none) -> Power DDR4 SODIMM
