File: fpga_candelabra/fmc_hpc.kicad_sch (KiCad schematic)
At the start: 1 part, among them J5 Samtec_ASP-134486-01

Commit message: candelabra: add i-pex extension ports, remove FMC1
* update bank/mgt allocation
* add basic pcb floorplanning

Signed-off-by: Yichuan Gao <gaoyichuan000@gmail.com>
Parts:
- added FM1: FMC_Outline_SingleWidth, CHIPSAlliance_Connector:FMC_Module_Outline, symbol CHIPSAlliance_Mechanical:FMC_Outline_SingleWidth
- J5: footprint (none) -> CHIPSAlliance_Connector:Samtec_FMC_ASP-134486-01_10x40_P1.27mm_Vertical
- J5: footprint Connector_Samtec:Samtec_FMC_ASP-134486-01_10x40_P1.27mm_Vertical -> CHIPSAlliance_Connector:Samtec_FMC_ASP-134486-01_10x40_P1.27mm_Vertical
Connections:
- net Earth: now also FM1.MH
- net FMC.PG_C2M renamed PG_C2M
