File: fpga_candelabra/fpga_candelabra.kicad_pcb (KiCad board)
At the start: 8 copper layers, 0 parts

Commit message: fpga_candelabra: reorganize fpga io and mgt by SLR
- Rename sch sheets
- Add prelimary DDR and PCIE Bank/Quad allocation

Signed-off-by: Yichuan Gao <gaoyichuan000@gmail.com>
Parts:
- added C1: 2.2nF, Capacitor_SMD:C_0402_1005Metric, F.Cu at (128.6, 112.2)
- added C10: 22uF 25V, Capacitor_SMD:C_1206_3216Metric, F.Cu at (92.9, 81.8)
- added C100: 4.7uF 10V, Capacitor_SMD:C_0402_1005Metric, F.Cu at (136.2, 42.9)
- added C101: 100nF, Capacitor_SMD:C_0402_1005Metric, F.Cu at (136.2, 44.9)
- added C102: 22uF 25V, Capacitor_SMD:C_1206_3216Metric, F.Cu at (123.3, 42.0)
- added C103: 100nF, Capacitor_SMD:C_0402_1005Metric, F.Cu at (136.2, 46.9)
- added C104: 2.2nF, Capacitor_SMD:C_0402_1005Metric, F.Cu at (139.9, 74.4)
- added C105: 4.7uF 10V, Capacitor_SMD:C_0402_1005Metric, F.Cu at (139.9, 76.4)
- added C106: 4.7uF 10V, Capacitor_SMD:C_0402_1005Metric, F.Cu at (139.9, 78.4)
- added C107: 100nF, Capacitor_SMD:C_0402_1005Metric, F.Cu at (139.9, 80.3)
- added C108: 22uF 25V, Capacitor_SMD:C_1206_3216Metric, F.Cu at (141.3, 86.9)
- added C109: 100nF, Capacitor_SMD:C_0402_1005Metric, F.Cu at (139.9, 82.3)
- added C11: 1uF, Capacitor_SMD:C_0402_1005Metric, F.Cu at (131.5, 112.2)
- added C110: 2.2nF, Capacitor_SMD:C_0402_1005Metric, F.Cu at (139.9, 84.3)
- added C111: 4.7uF 10V, Capacitor_SMD:C_0402_1005Metric, F.Cu at (142.8, 74.4)
- added C112: 4.7uF 10V, Capacitor_SMD:C_0402_1005Metric, F.Cu at (142.8, 76.4)
- added C113: 100nF, Capacitor_SMD:C_0402_1005Metric, F.Cu at (142.8, 78.4)
- added C114: 22uF 25V, Capacitor_SMD:C_1206_3216Metric, F.Cu at (141.3, 90.3)
- added C115: 100nF, Capacitor_SMD:C_0402_1005Metric, F.Cu at (142.8, 80.3)
- added C116: 100nF, Capacitor_SMD:C_0402_1005Metric, F.Cu at (142.8, 82.3)
- added C117: 27pF, Capacitor_SMD:C_0402_1005Metric, F.Cu at (59.6, 146.4)
- added C118: 27pF, Capacitor_SMD:C_0402_1005Metric, F.Cu at (59.6, 148.4)
- added C119: 100nF, Capacitor_SMD:C_0402_1005Metric, F.Cu at (59.6, 150.3)
- added C12: 4.7uF 10V, Capacitor_SMD:C_0402_1005Metric, F.Cu at (131.5, 114.2)
- added C120: 100nF, Capacitor_SMD:C_0402_1005Metric, F.Cu at (62.5, 142.4)
- added C121: 1uF, Capacitor_SMD:C_0402_1005Metric, F.Cu at (62.5, 144.4)
- added C122: 100nF, Capacitor_SMD:C_0402_1005Metric, F.Cu at (62.5, 146.4)
- added C123: 100nF, Capacitor_SMD:C_0402_1005Metric, F.Cu at (62.5, 148.4)
- added C124: 100nF, Capacitor_SMD:C_0402_1005Metric, F.Cu at (62.5, 150.3)
- added C125: 100nF, Capacitor_SMD:C_0402_1005Metric, F.Cu at (65.3, 142.4)
- added C126: 100nF, Capacitor_SMD:C_0402_1005Metric, F.Cu at (65.3, 144.4)
- added C127: 100nF, Capacitor_SMD:C_0402_1005Metric, F.Cu at (65.3, 146.4)
- added C128: 100nF, Capacitor_SMD:C_0402_1005Metric, F.Cu at (65.3, 148.4)
- added C129: 100nF, Capacitor_SMD:C_0402_1005Metric, F.Cu at (142.8, 98.1)
- added C13: 1uF, Capacitor_SMD:C_0402_1005Metric, F.Cu at (131.5, 116.1)
- added C130: 470nF, Capacitor_SMD:C_0402_1005Metric, F.Cu at (142.8, 100.0)
- added C131: 470nF, Capacitor_SMD:C_0402_1005Metric, F.Cu at (142.8, 102.0)
- added C132: 10uF 6.3V, Capacitor_SMD:C_0402_1005Metric, F.Cu at (112.5, 130.0)
- added C133: 10uF 6.3V, Capacitor_SMD:C_0402_1005Metric, F.Cu at (112.5, 131.9)
- added C134: 10uF 6.3V, Capacitor_SMD:C_0402_1005Metric, F.Cu at (112.5, 133.9)
- added C135: 10uF 6.3V, Capacitor_SMD:C_0402_1005Metric, F.Cu at (112.5, 135.9)
- added C136: 10uF 6.3V, Capacitor_SMD:C_0402_1005Metric, F.Cu at (112.5, 137.9)
- added C137: 10uF 6.3V, Capacitor_SMD:C_0402_1005Metric, F.Cu at (112.5, 139.8)
- added C138: 10uF 6.3V, Capacitor_SMD:C_0402_1005Metric, F.Cu at (112.5, 141.8)
- added C139: 10uF 6.3V, Capacitor_SMD:C_0402_1005Metric, F.Cu at (112.5, 143.8)
- added C14: 100uF 6.3V, Capacitor_SMD:C_1206_3216Metric, F.Cu at (92.9, 85.2)
- added C140: 10uF 6.3V, Capacitor_SMD:C_0402_1005Metric, F.Cu at (115.3, 130.0)
- added C141: 10uF 6.3V, Capacitor_SMD:C_0402_1005Metric, F.Cu at (115.3, 131.9)
- added C142: 10uF 6.3V, Capacitor_SMD:C_0402_1005Metric, F.Cu at (115.3, 133.9)
- added C143: 10uF 6.3V, Capacitor_SMD:C_0402_1005Metric, F.Cu at (115.3, 135.9)
- added C144: 10uF 6.3V, Capacitor_SMD:C_0402_1005Metric, F.Cu at (115.3, 137.9)
- added C145: 10uF 6.3V, Capacitor_SMD:C_0402_1005Metric, F.Cu at (115.3, 139.8)
- added C146: 10uF 6.3V, Capacitor_SMD:C_0402_1005Metric, F.Cu at (115.3, 141.8)
- added C147: 10uF 6.3V, Capacitor_SMD:C_0402_1005Metric, F.Cu at (115.3, 143.8)
- added C148: 100uF 6.3V, Capacitor_SMD:C_1206_3216Metric, F.Cu at (102.5, 130.7)
- added C149: 100uF 6.3V, Capacitor_SMD:C_1206_3216Metric, F.Cu at (102.5, 134.0)
- added C15: 100uF 6.3V, Capacitor_SMD:C_1206_3216Metric, F.Cu at (92.9, 88.5)
- added C150: 100uF 6.3V, Capacitor_SMD:C_1206_3216Metric, F.Cu at (102.5, 137.4)
- added C151: 100uF 6.3V, Capacitor_SMD:C_1206_3216Metric, F.Cu at (102.5, 140.7)
- added C152: 100uF 6.3V, Capacitor_SMD:C_1206_3216Metric, F.Cu at (102.5, 144.1)
- added C153: 100uF 6.3V, Capacitor_SMD:C_1206_3216Metric, F.Cu at (102.5, 147.4)
- added C154: 100uF 6.3V, Capacitor_SMD:C_1206_3216Metric, F.Cu at (108.2, 130.7)
- added C155: 100uF 6.3V, Capacitor_SMD:C_1206_3216Metric, F.Cu at (108.2, 134.0)
- added C156: 100uF 6.3V, Capacitor_SMD:C_1206_3216Metric, F.Cu at (108.2, 137.4)
- added C157: 100uF 6.3V, Capacitor_SMD:C_1206_3216Metric, F.Cu at (108.2, 140.7)
- added C158: 100uF 6.3V, Capacitor_SMD:C_1206_3216Metric, F.Cu at (108.2, 144.1)
- added C159: 330uF 2.5V, Capacitor_SMD:C_1210_3225Metric, F.Cu at (96.9, 131.1)
- added C16: 100uF 6.3V, Capacitor_SMD:C_1206_3216Metric, F.Cu at (92.9, 91.9)
- added C160: 47uF 6.3V, Capacitor_SMD:C_0603_1608Metric, F.Cu at (92.1, 130.2)
- added C161: 47uF 6.3V, Capacitor_SMD:C_0603_1608Metric, F.Cu at (92.1, 132.8)
- added C162: 47uF 6.3V, Capacitor_SMD:C_0603_1608Metric, F.Cu at (92.1, 135.3)
- added C163: 47uF 6.3V, Capacitor_SMD:C_0603_1608Metric, F.Cu at (92.1, 137.8)
- added C164: 47uF 6.3V, Capacitor_SMD:C_0603_1608Metric, F.Cu at (92.1, 140.3)
- added C165: 47uF 6.3V, Capacitor_SMD:C_0603_1608Metric, F.Cu at (92.1, 142.8)
- added C166: 330uF 2.5V, Capacitor_SMD:C_1210_3225Metric, F.Cu at (96.9, 135.4)
- added C167: 330uF 2.5V, Capacitor_SMD:C_1210_3225Metric, F.Cu at (96.9, 139.6)
- added C168: 330uF 2.5V, Capacitor_SMD:C_1210_3225Metric, F.Cu at (96.9, 143.9)
- added C169: 330uF 2.5V, Capacitor_SMD:C_1210_3225Metric, F.Cu at (96.9, 148.1)
- added C17: 100uF 6.3V, Capacitor_SMD:C_1206_3216Metric, F.Cu at (92.9, 95.2)
- added C170: 22uF 25V, Capacitor_SMD:C_1206_3216Metric, F.Cu at (35.3, 146.1)
- added C171: 22uF 25V, Capacitor_SMD:C_1206_3216Metric, F.Cu at (123.3, 45.4)
- added C172: 47uF 6.3V, Capacitor_SMD:C_0603_1608Metric, F.Cu at (92.1, 145.3)
- added C173: 10uF 6.3V, Capacitor_SMD:C_0402_1005Metric, F.Cu at (118.2, 130.0)
- added C174: 10uF 6.3V, Capacitor_SMD:C_0402_1005Metric, F.Cu at (118.2, 131.9)
- added C175: 47uF 6.3V, Capacitor_SMD:C_0603_1608Metric, F.Cu at (92.1, 147.8)
- added C176: 47uF 6.3V, Capacitor_SMD:C_0603_1608Metric, F.Cu at (92.1, 150.3)
- added C177: 10uF 6.3V, Capacitor_SMD:C_0402_1005Metric, F.Cu at (118.2, 133.9)
- added C178: 10uF 6.3V, Capacitor_SMD:C_0402_1005Metric, F.Cu at (118.2, 135.9)
- added C179: 4.7uF 10V, Capacitor_SMD:C_0402_1005Metric, F.Cu at (118.2, 137.9)
- added C18: 100uF 6.3V, Capacitor_SMD:C_1206_3216Metric, F.Cu at (92.9, 98.6)
- added C180: 4.7uF 10V, Capacitor_SMD:C_0402_1005Metric, F.Cu at (118.2, 139.8)
- added C181: 4.7uF 10V, Capacitor_SMD:C_0402_1005Metric, F.Cu at (118.2, 141.8)
- added C182: 4.7uF 10V, Capacitor_SMD:C_0402_1005Metric, F.Cu at (118.2, 143.8)
- added C183: 4.7uF 10V, Capacitor_SMD:C_0402_1005Metric, F.Cu at (121.1, 130.0)
- added C184: 4.7uF 10V, Capacitor_SMD:C_0402_1005Metric, F.Cu at (121.1, 131.9)
- added C185: 4.7uF 10V, Capacitor_SMD:C_0402_1005Metric, F.Cu at (121.1, 133.9)
- added C186: 4.7uF 10V, Capacitor_SMD:C_0402_1005Metric, F.Cu at (121.1, 135.9)
- added C187: 4.7uF 10V, Capacitor_SMD:C_0402_1005Metric, F.Cu at (121.1, 137.9)
- added C188: 4.7uF 10V, Capacitor_SMD:C_0402_1005Metric, F.Cu at (121.1, 139.8)
- added C189: 4.7uF 10V, Capacitor_SMD:C_0402_1005Metric, F.Cu at (121.1, 141.8)
- added C19: 100uF 6.3V, Capacitor_SMD:C_1206_3216Metric, F.Cu at (92.9, 101.9)
- added C190: 4.7uF 10V, Capacitor_SMD:C_0402_1005Metric, F.Cu at (121.1, 143.8)
- added C191: 100nF, Capacitor_SMD:C_0402_1005Metric, F.Cu at (136.9, 141.6)
- added C192: 1nF, Capacitor_SMD:C_0402_1005Metric, F.Cu at (136.9, 143.6)
- added C193: 100uF 6.3V, Capacitor_SMD:C_1206_3216Metric, F.Cu at (132.6, 130.7)
- added C194: 100uF 6.3V, Capacitor_SMD:C_1206_3216Metric, F.Cu at (132.6, 134.0)
- added C195: 100nF, Capacitor_SMD:C_0402_1005Metric, F.Cu at (136.9, 145.6)
- added C196: 22uF 25V, Capacitor_SMD:C_1206_3216Metric, F.Cu at (132.6, 137.4)
- added C197: 22uF 25V, Capacitor_SMD:C_1206_3216Metric, F.Cu at (132.6, 140.7)
- added C198: 1uF, Capacitor_SMD:C_0402_1005Metric, F.Cu at (136.9, 147.5)
- added C199: 4.7uF 10V, Capacitor_SMD:C_0402_1005Metric, F.Cu at (136.9, 149.5)
- added C2: 1nF, Capacitor_SMD:C_0402_1005Metric, F.Cu at (128.6, 114.2)
- added C20: 1uF, Capacitor_SMD:C_0402_1005Metric, F.Cu at (131.5, 118.1)
- added C200: 4.7uF 10V, Capacitor_SMD:C_0402_1005Metric, F.Cu at (139.8, 141.6)
- added C201: 4.7uF 10V, Capacitor_SMD:C_0402_1005Metric, F.Cu at (139.8, 143.6)
- added C202: 4.7uF 10V, Capacitor_SMD:C_0402_1005Metric, F.Cu at (139.8, 145.6)
- added C203: 1uF, Capacitor_SMD:C_0402_1005Metric, F.Cu at (139.8, 147.5)
- added C204: 2.2nF, Capacitor_SMD:C_0402_1005Metric, F.Cu at (139.8, 149.5)
- added C205: 4.7uF 10V, Capacitor_SMD:C_0402_1005Metric, F.Cu at (142.6, 141.6)
- added C206: 4.7uF 10V, Capacitor_SMD:C_0402_1005Metric, F.Cu at (142.6, 143.6)
- added C207: 100nF, Capacitor_SMD:C_0402_1005Metric, F.Cu at (142.6, 145.6)
- added C208: 22uF 25V, Capacitor_SMD:C_1206_3216Metric, F.Cu at (132.6, 144.1)
- added C209: 100nF, Capacitor_SMD:C_0402_1005Metric, F.Cu at (142.6, 147.5)
- added C21: 1uF, Capacitor_SMD:C_0402_1005Metric, F.Cu at (131.5, 120.1)
- added C210: 10uF 6.3V, Capacitor_SMD:C_0402_1005Metric, F.Cu at (33.9, 58.6)
- added C211: 10uF 6.3V, Capacitor_SMD:C_0402_1005Metric, F.Cu at (33.9, 60.6)
- added C212: 10uF 6.3V, Capacitor_SMD:C_0402_1005Metric, F.Cu at (33.9, 62.6)
- added C213: 10uF 6.3V, Capacitor_SMD:C_0402_1005Metric, F.Cu at (33.9, 64.5)
- added C214: 10uF 6.3V, Capacitor_SMD:C_0402_1005Metric, F.Cu at (33.9, 66.5)
- added C215: 100nF, Capacitor_SMD:C_0402_1005Metric, F.Cu at (33.9, 68.5)
- added C216: 100nF, Capacitor_SMD:C_0402_1005Metric, F.Cu at (33.9, 70.5)
- added C22: 100nF, Capacitor_SMD:C_0402_1005Metric, F.Cu at (131.5, 122.0)
- added C23: 4.7nF, Capacitor_SMD:C_0402_1005Metric, F.Cu at (131.5, 124.0)
- added C24: 100uF 6.3V, Capacitor_SMD:C_1206_3216Metric, F.Cu at (98.5, 75.1)
- added C25: 22uF 25V, Capacitor_SMD:C_1206_3216Metric, F.Cu at (98.5, 78.5)
- added C26: 100uF 6.3V, Capacitor_SMD:C_1206_3216Metric, F.Cu at (98.5, 81.8)
- added C27: 22uF 25V, Capacitor_SMD:C_1206_3216Metric, F.Cu at (98.5, 85.2)
- added C28: 100uF 6.3V, Capacitor_SMD:C_1206_3216Metric, F.Cu at (98.5, 88.5)
- added C29: 22uF 25V, Capacitor_SMD:C_1206_3216Metric, F.Cu at (98.5, 91.9)
- added C3: 12pF, Capacitor_SMD:C_0402_1005Metric, F.Cu at (128.6, 116.1)
- added C30: 100uF 6.3V, Capacitor_SMD:C_1206_3216Metric, F.Cu at (98.5, 95.2)
- added C31: 100uF 6.3V, Capacitor_SMD:C_1206_3216Metric, F.Cu at (98.5, 98.6)
- added C32: 100uF 6.3V, Capacitor_SMD:C_1206_3216Metric, F.Cu at (98.5, 101.9)
- added C33: 1uF, Capacitor_SMD:C_0402_1005Metric, F.Cu at (134.4, 112.2)
- added C34: 100nF, Capacitor_SMD:C_0402_1005Metric, F.Cu at (134.4, 114.2)
- added C35: 4.7nF, Capacitor_SMD:C_0402_1005Metric, F.Cu at (134.4, 116.1)
- added C36: 100uF 6.3V, Capacitor_SMD:C_1206_3216Metric, F.Cu at (104.2, 75.1)
- added C37: 22uF 25V, Capacitor_SMD:C_1206_3216Metric, F.Cu at (104.2, 78.5)
- added C38: 100uF 6.3V, Capacitor_SMD:C_1206_3216Metric, F.Cu at (104.2, 81.8)
- added C39: 22uF 25V, Capacitor_SMD:C_1206_3216Metric, F.Cu at (104.2, 85.2)
- added C4: 220nF, Capacitor_SMD:C_0402_1005Metric, F.Cu at (128.6, 118.1)
- added C40: 100uF 6.3V, Capacitor_SMD:C_1206_3216Metric, F.Cu at (104.2, 88.5)
- added C41: 22uF 25V, Capacitor_SMD:C_1206_3216Metric, F.Cu at (104.2, 91.9)
- added C42: 100uF 6.3V, Capacitor_SMD:C_1206_3216Metric, F.Cu at (104.2, 95.2)
- added C43: 100uF 6.3V, Capacitor_SMD:C_1206_3216Metric, F.Cu at (104.2, 98.6)
- added C44: 100uF 6.3V, Capacitor_SMD:C_1206_3216Metric, F.Cu at (104.2, 101.9)
- added C45: 1uF, Capacitor_SMD:C_0402_1005Metric, F.Cu at (134.4, 118.1)
- added C46: 100nF, Capacitor_SMD:C_0402_1005Metric, F.Cu at (134.4, 120.1)
- added C47: 4.7nF, Capacitor_SMD:C_0402_1005Metric, F.Cu at (134.4, 122.0)
- added C48: 100uF 6.3V, Capacitor_SMD:C_1206_3216Metric, F.Cu at (109.8, 75.1)
- added C49: 22uF 25V, Capacitor_SMD:C_1206_3216Metric, F.Cu at (109.8, 78.5)
- added C5: 100nF, Capacitor_SMD:C_0402_1005Metric, F.Cu at (128.6, 120.1)
- added C50: 100uF 6.3V, Capacitor_SMD:C_1206_3216Metric, F.Cu at (109.8, 81.8)
- added C51: 22uF 25V, Capacitor_SMD:C_1206_3216Metric, F.Cu at (109.8, 85.2)
- added C52: 100uF 6.3V, Capacitor_SMD:C_1206_3216Metric, F.Cu at (109.8, 88.5)
- added C53: 22uF 25V, Capacitor_SMD:C_1206_3216Metric, F.Cu at (109.8, 91.9)
- added C54: 100uF 6.3V, Capacitor_SMD:C_1206_3216Metric, F.Cu at (109.8, 95.2)
- added C55: 100uF 6.3V, Capacitor_SMD:C_1206_3216Metric, F.Cu at (109.8, 98.6)
- added C56: 100uF 6.3V, Capacitor_SMD:C_1206_3216Metric, F.Cu at (109.8, 101.9)
- added C57: 470uF 2V, Capacitor_Tantalum_SMD:CP_EIA-7343-20_Kemet-V, F.Cu at (95.0, 106.5)
- added C58: 470uF 2V, Capacitor_Tantalum_SMD:CP_EIA-7343-20_Kemet-V, F.Cu at (95.0, 112.4)
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Other:
- board outline added: 70.2 x 1.7 mm

Commit message: fpga_candelabra: pcb basic floorplan
Parts:
- added C217: 100nF, Capacitor_SMD:C_0402_1005Metric, F.Cu at (266.3, 68.9)
- added C218: 100nF, Capacitor_SMD:C_0402_1005Metric, F.Cu at (266.3, 70.9)
- added C219: 100nF, Capacitor_SMD:C_0402_1005Metric, F.Cu at (262.5, 82.4)
- added C220: 100nF, Capacitor_SMD:C_0402_1005Metric, F.Cu at (266.3, 72.8)
- added C221: 4.7pF, Capacitor_SMD:C_0402_1005Metric, F.Cu at (51.8, 189.7)
- added C222: 4.7pF, Capacitor_SMD:C_0402_1005Metric, F.Cu at (51.8, 191.7)
- added C223: 10uF 6.3V, Capacitor_SMD:C_0402_1005Metric, F.Cu at (51.8, 193.6)
- added C224: 22nF, Capacitor_SMD:C_0402_1005Metric, F.Cu at (51.8, 195.6)
- added C225: 100nF, Capacitor_SMD:C_0402_1005Metric, F.Cu at (51.8, 197.6)
- added C226: 100nF, Capacitor_SMD:C_0402_1005Metric, F.Cu at (51.8, 199.5)
- added C227: 100nF, Capacitor_SMD:C_0402_1005Metric, F.Cu at (54.7, 189.7)
- added C228: 100nF, Capacitor_SMD:C_0402_1005Metric, F.Cu at (54.7, 191.7)
- added C229: 100nF, Capacitor_SMD:C_0402_1005Metric, F.Cu at (54.7, 193.6)
- added C230: 100nF, Capacitor_SMD:C_0402_1005Metric, F.Cu at (54.7, 195.6)
- added C231: 100nF, Capacitor_SMD:C_0402_1005Metric, F.Cu at (54.7, 197.6)
- added C232: 100nF, Capacitor_SMD:C_0402_1005Metric, F.Cu at (54.7, 199.5)
- added C233: 100nF, Capacitor_SMD:C_0402_1005Metric, F.Cu at (57.6, 189.7)
- added C234: 100nF, Capacitor_SMD:C_0402_1005Metric, F.Cu at (57.6, 191.7)
- added C235: 100nF, Capacitor_SMD:C_0402_1005Metric, F.Cu at (57.6, 193.6)
- added C236: 100nF, Capacitor_SMD:C_0402_1005Metric, F.Cu at (57.6, 195.6)
- added C237: 100nF, Capacitor_SMD:C_0402_1005Metric, F.Cu at (57.6, 197.6)
- added C238: 220nF, Capacitor_SMD:C_0402_1005Metric, B.Cu at (62.8, 168.6)
- added C239: 220nF, Capacitor_SMD:C_0402_1005Metric, B.Cu at (63.7, 168.6)
- added C240: 220nF, Capacitor_SMD:C_0402_1005Metric, B.Cu at (67.7, 168.6)
- added C241: 220nF, Capacitor_SMD:C_0402_1005Metric, B.Cu at (68.7, 168.6)
- added C242: 220nF, Capacitor_SMD:C_0402_1005Metric, B.Cu at (71.8, 168.6)
- added C243: 220nF, Capacitor_SMD:C_0402_1005Metric, B.Cu at (72.7, 168.6)
- added C244: 220nF, Capacitor_SMD:C_0402_1005Metric, B.Cu at (75.7, 168.6)
- added C245: 220nF, Capacitor_SMD:C_0402_1005Metric, B.Cu at (76.7, 168.6)
- added C246: 220nF, Capacitor_SMD:C_0402_1005Metric, B.Cu at (81.7, 168.6)
- added C247: 220nF, Capacitor_SMD:C_0402_1005Metric, B.Cu at (82.7, 168.6)
- added C248: 220nF, Capacitor_SMD:C_0402_1005Metric, B.Cu at (85.7, 168.6)
- added C249: 220nF, Capacitor_SMD:C_0402_1005Metric, B.Cu at (86.7, 168.6)
- added C250: 220nF, Capacitor_SMD:C_0402_1005Metric, B.Cu at (89.7, 168.6)
- added C251: 220nF, Capacitor_SMD:C_0402_1005Metric, B.Cu at (90.7, 168.6)
- added C252: 220nF, Capacitor_SMD:C_0402_1005Metric, B.Cu at (93.7, 168.6)
- added C253: 220nF, Capacitor_SMD:C_0402_1005Metric, B.Cu at (94.7, 168.6)
- added C254: 220nF, Capacitor_SMD:C_0402_1005Metric, B.Cu at (98.7, 168.6)
- added C255: 220nF, Capacitor_SMD:C_0402_1005Metric, B.Cu at (99.7, 168.6)
- added C256: 220nF, Capacitor_SMD:C_0402_1005Metric, B.Cu at (102.7, 168.6)
- added C257: 220nF, Capacitor_SMD:C_0402_1005Metric, B.Cu at (103.7, 168.6)
- added C258: 220nF, Capacitor_SMD:C_0402_1005Metric, B.Cu at (106.7, 168.6)
- added C259: 220nF, Capacitor_SMD:C_0402_1005Metric, B.Cu at (107.7, 168.6)
- added C260: 220nF, Capacitor_SMD:C_0402_1005Metric, B.Cu at (110.7, 168.6)
- added C261: 220nF, Capacitor_SMD:C_0402_1005Metric, B.Cu at (111.7, 168.6)
- added C262: 220nF, Capacitor_SMD:C_0402_1005Metric, B.Cu at (114.7, 168.6)
- added C263: 220nF, Capacitor_SMD:C_0402_1005Metric, B.Cu at (115.7, 168.6)
- added C264: 220nF, Capacitor_SMD:C_0402_1005Metric, B.Cu at (118.7, 168.6)
- added C265: 220nF, Capacitor_SMD:C_0402_1005Metric, B.Cu at (119.7, 168.6)
- added C266: 220nF, Capacitor_SMD:C_0402_1005Metric, B.Cu at (122.7, 168.6)
- added C267: 220nF, Capacitor_SMD:C_0402_1005Metric, B.Cu at (123.7, 168.6)
- added C268: 220nF, Capacitor_SMD:C_0402_1005Metric, B.Cu at (126.7, 168.6)
- added C269: 220nF, Capacitor_SMD:C_0402_1005Metric, B.Cu at (127.7, 168.6)
- added C270: 100nF, Capacitor_SMD:C_0402_1005Metric, B.Cu at (59.7, 168.6)
- added C271: 100nF, Capacitor_SMD:C_0402_1005Metric, B.Cu at (60.6, 168.6)
- added C272: 22uF 25V, Capacitor_SMD:C_1206_3216Metric, F.Cu at (155.1, 99.8)
- added C273: 22uF 25V, Capacitor_SMD:C_1206_3216Metric, F.Cu at (155.1, 103.2)
- added C274: 22nF, Capacitor_SMD:C_0402_1005Metric, F.Cu at (150.9, 99.2)
- added C275: 1uF, Capacitor_SMD:C_0402_1005Metric, F.Cu at (150.9, 101.1)
- added C276: 47pF, Capacitor_SMD:C_0402_1005Metric, F.Cu at (150.9, 103.1)
- added C277: 100nF, Capacitor_SMD:C_0402_1005Metric, F.Cu at (150.9, 105.1)
- added C278: 100uF 6.3V, Capacitor_SMD:C_1206_3216Metric, F.Cu at (155.1, 106.5)
- added C280: 220pF, Capacitor_SMD:C_0402_1005Metric, F.Cu at (150.9, 107.0)
- added C281: 100nF, Capacitor_SMD:C_0402_1005Metric, F.Cu at (150.9, 109.0)
- added F1: 16V 1.5A Polyfuse, Resistor_SMD:R_1206_3216Metric, F.Cu at (146.6, 99.8)
- added F2: 16V 1.5A Polyfuse, Resistor_SMD:R_1206_3216Metric, F.Cu at (146.6, 103.1)
- added F3: 6V 4A Polyfuse, Resistor_SMD:R_1206_3216Metric, F.Cu at (146.6, 106.4)
- added F4: 6V 4A Polyfuse, Resistor_SMD:R_1206_3216Metric, F.Cu at (146.6, 109.7)
- added F5: 6V 4A Polyfuse, Resistor_SMD:R_1206_3216Metric, F.Cu at (146.6, 113.0)
- added F6: 6V 4A Polyfuse, Resistor_SMD:R_1206_3216Metric, F.Cu at (146.6, 116.3)
- added J3: Bus_PCI_Express_x16, Connector_PCBEdge:BUS_PCIexpress_x16, F.Cu at (45.7, 174.9)
- added J4: Molex 45558-0003, Connector_Molex:Molex_Mini-Fit_Jr_5569-06A2_2x03_P4.20mm_Horizontal, F.Cu at (36.3, 203.6)
- added J5: Samtec_ASP-134486-01, Connector_Samtec:Samtec_FMC_ASP-134486-01_10x40_P1.27mm_Vertical, F.Cu at (111.0, 72.4)
- added J6: Samtec_ASP-134486-01, Connector_Samtec:Samtec_FMC_ASP-134486-01_10x40_P1.27mm_Vertical, F.Cu at (111.1, 133.8)
- added R100: 1k, Resistor_SMD:R_0402_1005Metric, B.Cu at (26.6, 87.1)
- added R101: 1k, Resistor_SMD:R_0402_1005Metric, B.Cu at (26.6, 89.1)
- added R102: 1k, Resistor_SMD:R_0402_1005Metric, B.Cu at (26.6, 91.1)
- added R103: 240R 1%, Resistor_SMD:R_0402_1005Metric, B.Cu at (26.6, 93.1)
- added R104: 240R 1%, Resistor_SMD:R_0402_1005Metric, B.Cu at (26.6, 95.1)
- added R105: 240R 1%, Resistor_SMD:R_0402_1005Metric, B.Cu at (26.6, 97.1)
- added R106: 100R, Resistor_SMD:R_0402_1005Metric, F.Cu at (51.9, 205.5)
- added R107: 100R, Resistor_SMD:R_0402_1005Metric, F.Cu at (51.9, 207.4)
- added R108: 100R, Resistor_SMD:R_0402_1005Metric, F.Cu at (51.9, 209.4)
- added R109: 1k, Resistor_SMD:R_0402_1005Metric, F.Cu at (65.7, 199.0)
- added R110: 1k, Resistor_SMD:R_0402_1005Metric, F.Cu at (65.7, 201.0)
- added R111: 0R, Resistor_SMD:R_0402_1005Metric, F.Cu at (98.8, 47.4)
- added R112: 0R, Resistor_SMD:R_0402_1005Metric, F.Cu at (100.8, 47.4)
- added R113: 0R, Resistor_SMD:R_0402_1005Metric, F.Cu at (98.6, 159.8)
- added R114: 0R, Resistor_SMD:R_0402_1005Metric, F.Cu at (100.5, 159.8)
- added R115: 100k, Resistor_SMD:R_0402_1005Metric, F.Cu at (150.9, 111.0)
- added R116: 22k, Resistor_SMD:R_0402_1005Metric, F.Cu at (150.9, 113.0)
- added R87: 100k, Resistor_SMD:R_0402_1005Metric, F.Cu at (257.6, 68.9)
- added R88: 2.2k, Resistor_SMD:R_0402_1005Metric, F.Cu at (257.6, 70.9)
- added R89: 2.2k, Resistor_SMD:R_0402_1005Metric, F.Cu at (257.6, 72.9)
- added R90: 2.2k, Resistor_SMD:R_0402_1005Metric, F.Cu at (260.5, 68.9)
- added R91: 2.2k, Resistor_SMD:R_0402_1005Metric, F.Cu at (260.5, 70.9)
- added R92: 10k, Resistor_SMD:R_0402_1005Metric, F.Cu at (260.5, 72.9)
- added R93: 10k, Resistor_SMD:R_0402_1005Metric, F.Cu at (263.4, 68.9)
- added R94: 100R, Resistor_SMD:R_0402_1005Metric, F.Cu at (257.6, 80.4)
- added R95: 330R, Resistor_SMD:R_0402_1005Metric, F.Cu at (257.6, 82.4)
- added R96: 10k, Resistor_SMD:R_0402_1005Metric, F.Cu at (252.7, 82.9)
- added R97: 10k, Resistor_SMD:R_0402_1005Metric, F.Cu at (263.4, 70.9)
- added R98: 2.2k, Resistor_SMD:R_0402_1005Metric, F.Cu at (263.4, 72.9)
- added R99: 4.7k, Resistor_SMD:R_0402_1005Metric, F.Cu at (262.5, 80.4)
- added U21: PCA9306DC, Package_SO:VSSOP-8_2.3x2mm_P0.5mm, F.Cu at (259.1, 75.7)
- added U22: CDCM6208V1, Package_DFN_QFN:Texas_RGZ0048A_VQFN-48-1EP_7x7mm_P0.5mm_EP5.15x5.15mm, F.Cu at (63.7, 193.4)
- added Y2: NX3225GA 25MHz, Crystal:Crystal_SMD_3225-4Pin_3.2x2.5mm, F.Cu at (61.6, 200.2)
- C105, C106: value 4.7uF 10V -> 22uF 25V; footprint Capacitor_SMD:C_0402_1005Metric -> Capacitor_SMD:C_1206_3216Metric
- C107: value 100nF -> 10nF
- C108: value 22uF 25V -> 1uF; footprint Capacitor_SMD:C_1206_3216Metric -> Capacitor_SMD:C_0402_1005Metric
- C109: value 100nF -> 47pF
- C110: value 2.2nF -> 100nF
- C111: value 4.7uF 10V -> 2.2nF
- C112: value 4.7uF 10V -> 100uF 6.3V; footprint Capacitor_SMD:C_0402_1005Metric -> Capacitor_SMD:C_1206_3216Metric
- C113: value 100nF -> 100uF 6.3V; footprint Capacitor_SMD:C_0402_1005Metric -> Capacitor_SMD:C_1206_3216Metric
- C114: value 22uF 25V -> 100nF; footprint Capacitor_SMD:C_1206_3216Metric -> Capacitor_SMD:C_0402_1005Metric
- J1: value USB_C_Receptacle_USB2.0_14P -> TYPE-C-31-M-12
- L10, L11: value MWSA0402S-2R2MT -> MWSA1004S-2R2MT; footprint Inductor_SMD:L_Sunlord_MWSA0402S -> Inductor_SMD:L_Sunlord_MWSA1004S
- R56: value 27k -> 10k
- R57: value 56k -> 51k
- R58: value 10k -> 2.2k
- R60: value 10k -> 27k
- R61: value 10k -> 56k
- R62: value 56k -> 10k
- R63: value 27k -> 51k
- R64: value DNP/2.2k -> 1k
- R65: value DNP/2.2k -> DNP/10k
- R67, R68: value 10k -> 27R
- U11, U7: footprint Package_DFN_QFN:Texas_VQFN-RHL-20 -> CHIPSAlliance_Package_DFN_QFN:Texas_VQFN-RHL-14
- U14: value MCP4631-104E-ST -> TPS54821; footprint Package_SO:TSSOP-14_4.4x5mm_P0.65mm -> CHIPSAlliance_Package_DFN_QFN:Texas_VQFN-RHL-14
- U15: value TLV62130x -> MCP4017-104ELT; footprint CHIPSAlliance_Package_DFN_QFN:Texas_RGT0016C_VQFN-16-1EP_3x3mm_P0.5mm_EP1.68x1.68mm -> Package_TO_SOT_SMD:SOT-363_SC-70-6
- U16: value TLV62130x -> TPS54821; footprint CHIPSAlliance_Package_DFN_QFN:Texas_RGT0016C_VQFN-16-1EP_3x3mm_P0.5mm_EP1.68x1.68mm -> CHIPSAlliance_Package_DFN_QFN:Texas_VQFN-RHL-14
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Connections:
- net /DDR4 SODIMM/A0 renamed /DDR4.A0
- net /DDR4 SODIMM/A1 renamed /DDR4.A1
- net /DDR4 SODIMM/A10 renamed /DDR4.A10
- net /DDR4 SODIMM/A11 renamed /DDR4.A11
- net /DDR4 SODIMM/A12 renamed /DDR4.A12
- net /DDR4 SODIMM/A13 renamed /DDR4.A13
- net /DDR4 SODIMM/A14 renamed /DDR4.A14
- net /DDR4 SODIMM/A15 renamed /DDR4.A15
- net /DDR4 SODIMM/A16 renamed /DDR4.A16
- net /DDR4 SODIMM/A2 renamed /DDR4.A2
- net /DDR4 SODIMM/A3 renamed /DDR4.A3
- net /DDR4 SODIMM/A4 renamed /DDR4.A4
- net /DDR4 SODIMM/A5 renamed /DDR4.A5
- net /DDR4 SODIMM/A6 renamed /DDR4.A6
- net /DDR4 SODIMM/A7 renamed /DDR4.A7
- net /DDR4 SODIMM/A8 renamed /DDR4.A8
- net /DDR4 SODIMM/A9 renamed /DDR4.A9
- net /DDR4 SODIMM/ACT_n renamed /DDR4 SODIMM/DDR4.ACT_n
- net /DDR4 SODIMM/ALERT_n renamed /DDR4 SODIMM/DDR4.ALERT_n
- net /DDR4 SODIMM/BA0 renamed /DDR4.BA0
- net /DDR4 SODIMM/BA1 renamed /DDR4.BA1
- net /DDR4 SODIMM/BG0 renamed /DDR4.BG0
- net /DDR4 SODIMM/BG1 renamed /DDR4.BG1
- net /DDR4 SODIMM/CB0 renamed /DDR4.CB0
- net /DDR4 SODIMM/CB1 renamed /DDR4.CB1
- net /DDR4 SODIMM/CB2 renamed /DDR4.CB2
- net /DDR4 SODIMM/CB3 renamed /DDR4.CB3
- net /DDR4 SODIMM/CB4 renamed /DDR4.CB4
- net /DDR4 SODIMM/CB5 renamed /DDR4.CB5
- net /DDR4 SODIMM/CB6 renamed /DDR4.CB6
- net /DDR4 SODIMM/CB7 renamed /DDR4.CB7
- net /DDR4 SODIMM/CK0+ renamed /DDR4.CK0+
- net /DDR4 SODIMM/CK0- renamed /DDR4.CK0-
- net /DDR4 SODIMM/CK1+ renamed /DDR4.CK1+
- net /DDR4 SODIMM/CK1- renamed /DDR4.CK1-
- net /DDR4 SODIMM/CKE0 renamed /DDR4.CKE0
- net /DDR4 SODIMM/CKE1 renamed /DDR4.CKE1
- net /DDR4 SODIMM/CS0 renamed /DDR4.CS0
- net /DDR4 SODIMM/CS1 renamed /DDR4.CS1
- net /DDR4 SODIMM/CS2 renamed /DDR4.CS2
- net /DDR4 SODIMM/CS3 renamed /DDR4.CS3
- net /DDR4 SODIMM/DM0 renamed /DDR4.DM0
- net /DDR4 SODIMM/DM1 renamed /DDR4.DM1
- net /DDR4 SODIMM/DM2 renamed /DDR4.DM2
- net /DDR4 SODIMM/DM3 renamed /DDR4.DM3
- net /DDR4 SODIMM/DM4 renamed /DDR4.DM4
- net /DDR4 SODIMM/DM5 renamed /DDR4.DM5
- net /DDR4 SODIMM/DM6 renamed /DDR4.DM6
- net /DDR4 SODIMM/DM7 renamed /DDR4.DM7
- net /DDR4 SODIMM/DM8 renamed /DDR4.DM8
- net /DDR4 SODIMM/DQ0 renamed /DDR4.DQ0
- net /DDR4 SODIMM/DQ1 renamed /DDR4.DQ1
- net /DDR4 SODIMM/DQ10 renamed /DDR4.DQ10
- net /DDR4 SODIMM/DQ11 renamed /DDR4.DQ11
- net /DDR4 SODIMM/DQ12 renamed /DDR4.DQ12
- net /DDR4 SODIMM/DQ13 renamed /DDR4.DQ13
- net /DDR4 SODIMM/DQ14 renamed /DDR4.DQ14
- net /DDR4 SODIMM/DQ15 renamed /DDR4.DQ15
- net /DDR4 SODIMM/DQ16 renamed /DDR4.DQ16
- net /DDR4 SODIMM/DQ17 renamed /DDR4.DQ17
- net /DDR4 SODIMM/DQ18 renamed /DDR4.DQ18
- net /DDR4 SODIMM/DQ19 renamed /DDR4.DQ19
- net /DDR4 SODIMM/DQ2 renamed /DDR4.DQ2
- net /DDR4 SODIMM/DQ20 renamed /DDR4.DQ20
- net /DDR4 SODIMM/DQ21 renamed /DDR4.DQ21
- net /DDR4 SODIMM/DQ22 renamed /DDR4.DQ22
- net /DDR4 SODIMM/DQ23 renamed /DDR4.DQ23
- net /DDR4 SODIMM/DQ24 renamed /DDR4.DQ24
- net /DDR4 SODIMM/DQ25 renamed /DDR4.DQ25
- net /DDR4 SODIMM/DQ26 renamed /DDR4.DQ26
- net /DDR4 SODIMM/DQ27 renamed /DDR4.DQ27
- net /DDR4 SODIMM/DQ28 renamed /DDR4.DQ28
- net /DDR4 SODIMM/DQ29 renamed /DDR4.DQ29
- net /DDR4 SODIMM/DQ3 renamed /DDR4.DQ3
- net /DDR4 SODIMM/DQ30 renamed /DDR4.DQ30
- net /DDR4 SODIMM/DQ31 renamed /DDR4.DQ31
- net /DDR4 SODIMM/DQ32 renamed /DDR4.DQ32
- net /DDR4 SODIMM/DQ33 renamed /DDR4.DQ33
- net /DDR4 SODIMM/DQ34 renamed /DDR4.DQ34
- net /DDR4 SODIMM/DQ35 renamed /DDR4.DQ35
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Other:
- board size 70.2 x 1.7 mm -> 84.3 x 8.4 mm

Commit message: candelabra: add i-pex extension ports, remove FMC1
* update bank/mgt allocation
* add basic pcb floorplanning

Signed-off-by: Yichuan Gao <gaoyichuan000@gmail.com>
Parts:
- removed J6: Samtec_ASP-134486-01, Connector_Samtec:Samtec_FMC_ASP-134486-01_10x40_P1.27mm_Vertical
- removed R113, R114: 0R, Resistor_SMD:R_0402_1005Metric
- added C279: 100nF, Capacitor_SMD:C_0402_1005Metric, B.Cu at (24.3, 129.7)
- added C282: 22uF 25V, Capacitor_SMD:C_1206_3216Metric, B.Cu at (28.6, 130.4)
- added C283: 100nF, Capacitor_SMD:C_0402_1005Metric, B.Cu at (24.3, 131.7)
- added C284: 22uF 25V, Capacitor_SMD:C_1206_3216Metric, B.Cu at (28.6, 133.7)
- added C285: 100nF, Capacitor_SMD:C_0402_1005Metric, B.Cu at (24.3, 133.6)
- added C286: 22uF 25V, Capacitor_SMD:C_1206_3216Metric, B.Cu at (28.6, 137.1)
- added C287: 100nF, Capacitor_SMD:C_0402_1005Metric, B.Cu at (24.3, 135.6)
- added C288: 100nF, Capacitor_SMD:C_0402_1005Metric, B.Cu at (24.3, 137.6)
- added C289: 100nF, Capacitor_SMD:C_0402_1005Metric, B.Cu at (38.3, 154.0)
- added C290: 22uF 25V, Capacitor_SMD:C_1206_3216Metric, B.Cu at (31.1, 154.7)
- added C291: 100nF, Capacitor_SMD:C_0402_1005Metric, B.Cu at (38.3, 156.0)
- added C292: 100nF, Capacitor_SMD:C_0402_1005Metric, B.Cu at (38.3, 157.9)
- added C293: 100nF, Capacitor_SMD:C_0402_1005Metric, B.Cu at (38.3, 159.9)
- added C294: 22uF 25V, Capacitor_SMD:C_1206_3216Metric, B.Cu at (31.1, 158.0)
- added C295: 22uF 25V, Capacitor_SMD:C_1206_3216Metric, B.Cu at (31.1, 161.4)
- added C296: 22uF 25V, Capacitor_SMD:C_1206_3216Metric, B.Cu at (31.1, 164.7)
- added C297: 100nF, Capacitor_SMD:C_0402_1005Metric, B.Cu at (38.3, 161.9)
- added C298: 100nF, Capacitor_SMD:C_0402_1005Metric, B.Cu at (38.3, 163.8)
- added C299: 100nF, Capacitor_SMD:C_0402_1005Metric, B.Cu at (38.3, 165.8)
- added C300: 100nF, Capacitor_SMD:C_0402_1005Metric, B.Cu at (38.3, 167.8)
- added C301: 100nF, Capacitor_SMD:C_0402_1005Metric, B.Cu at (136.3, 55.6)
- added C302: 100nF, Capacitor_SMD:C_0402_1005Metric, B.Cu at (136.3, 57.5)
- added C303: 10uF 6.3V, Capacitor_SMD:C_0402_1005Metric, B.Cu at (182.5, 148.0)
- added C304: 47uF 6.3V, Capacitor_SMD:C_0603_1608Metric, B.Cu at (174.0, 147.5)
- added C305: 10uF 6.3V, Capacitor_SMD:C_0402_1005Metric, B.Cu at (185.5, 152.0)
- added C306: 10uF 6.3V, Capacitor_SMD:C_0402_1005Metric, B.Cu at (182.5, 158.0)
- added C307: 47uF 6.3V, Capacitor_SMD:C_0603_1608Metric, B.Cu at (174.0, 157.5)
- added FM1: FMC_Outline_SingleWidth, CHIPSAlliance_Connector:FMC_Module_Outline, F.Cu at (275.7, 117.1)
- added H1: M3.0, MountingHole:MountingHole_3.2mm_M3_DIN965, F.Cu at (163.5, 116.5)
- added H2: M3.0, MountingHole:MountingHole_3.2mm_M3_DIN965, F.Cu at (226.5, 116.5)
- added H3: M3.0, MountingHole:MountingHole_3.2mm_M3_DIN965, F.Cu at (226.5, 179.5)
- added H4: M3.0, MountingHole:MountingHole_3.2mm_M3_DIN965, F.Cu at (163.5, 179.5)
- added IPEX0: 20455-040E-76, CHIPSAlliance_Connector:I-PEX_20455-040E-76, F.Cu at (163.5, 102.6)
- added IPEX1: 20455-040E-76, CHIPSAlliance_Connector:I-PEX_20455-040E-76, F.Cu at (226.5, 102.6)
- added IPEX2: 20455-040E-76, CHIPSAlliance_Connector:I-PEX_20455-040E-76, B.Cu at (163.5, 102.6)
- added IPEX3: 20455-040E-76, CHIPSAlliance_Connector:I-PEX_20455-040E-76, B.Cu at (226.5, 102.6)
- added IPEX4: 20455-050E-76, CHIPSAlliance_Connector:I-PEX_20455-050E-76, F.Cu at (195.0, 102.6)
- added J7: QSFP+, CHIPSAlliance_Connector:Connector_QSFP_and_Cage, F.Cu at (92.7, 122.5)
- added J8: QSFP+, CHIPSAlliance_Connector:Connector_QSFP_and_Cage, F.Cu at (92.7, 146.5)
- added L14: SLM25201R0MIT, Inductor_SMD:L_1008_2520Metric, B.Cu at (33.9, 130.6)
- added L15: SLM25201R0MIT, Inductor_SMD:L_1008_2520Metric, B.Cu at (33.9, 134.3)
- added L16: SLM25201R0MIT, Inductor_SMD:L_1008_2520Metric, B.Cu at (33.9, 138.1)
- added L17: SLM25201R0MIT, Inductor_SMD:L_1008_2520Metric, B.Cu at (25.8, 154.9)
- added L18: SLM25201R0MIT, Inductor_SMD:L_1008_2520Metric, B.Cu at (25.8, 158.6)
- added L19: SLM25201R0MIT, Inductor_SMD:L_1008_2520Metric, B.Cu at (25.8, 162.4)
- added R117: 100k, Resistor_SMD:R_0402_1005Metric, B.Cu at (37.8, 129.7)
- added R118: 2.2k, Resistor_SMD:R_0402_1005Metric, B.Cu at (37.8, 131.7)
- added R119: 2.2k, Resistor_SMD:R_0402_1005Metric, B.Cu at (37.8, 133.7)
- added R120: 2.2k, Resistor_SMD:R_0402_1005Metric, B.Cu at (37.8, 135.7)
- added R121: 2.2k, Resistor_SMD:R_0402_1005Metric, B.Cu at (37.8, 137.7)
- added R122: 0R, Resistor_SMD:R_0402_1005Metric, B.Cu at (37.8, 139.7)
- added R123: 2.2k, Resistor_SMD:R_0402_1005Metric, B.Cu at (37.8, 141.6)
- added R124: 0R, Resistor_SMD:R_0402_1005Metric, B.Cu at (35.4, 154.0)
- added R125: 2.2k, Resistor_SMD:R_0402_1005Metric, B.Cu at (35.4, 156.0)
- added R126: 2.2k, Resistor_SMD:R_0402_1005Metric, B.Cu at (35.4, 158.0)
- added R127: 2.2k, Resistor_SMD:R_0402_1005Metric, B.Cu at (35.4, 160.0)
- added R128: 100k, Resistor_SMD:R_0402_1005Metric, B.Cu at (35.4, 162.0)
- added R129: 2.2k, Resistor_SMD:R_0402_1005Metric, B.Cu at (35.4, 163.9)
- added R130: 2.2k, Resistor_SMD:R_0402_1005Metric, B.Cu at (35.4, 165.9)
- added R131: DNP/0R, Resistor_SMD:R_0402_1005Metric, F.Cu at (244.0, 173.0)
- added R132: DNP/0R, Resistor_SMD:R_0402_1005Metric, F.Cu at (245.0, 173.0)
- added R133: 0R, Resistor_SMD:R_0402_1005Metric, F.Cu at (243.0, 173.0)
- added REF**: PCIexpress_bracket_full, PCIexpress:PCIexpress_bracket_full, F.Cu at (100.8, 200.7)
- added TP1: TestPoint_Small, TestPoint:TestPoint_Pad_D1.0mm, F.Cu at (252.8, 170.2)
- added TP2: TestPoint_Small, TestPoint:TestPoint_Pad_D1.0mm, F.Cu at (252.8, 155.0)
- added TP3: TestPoint_Small, TestPoint:TestPoint_Pad_D1.0mm, F.Cu at (252.8, 139.7)
- added TP4: TestPoint_Small, TestPoint:TestPoint_Pad_D1.0mm, F.Cu at (252.8, 124.4)
- added TP5: TestPoint_Small, TestPoint:TestPoint_Pad_D1.0mm, F.Cu at (250.5, 170.2)
- added TP6: TestPoint_Small, TestPoint:TestPoint_Pad_D1.0mm, F.Cu at (250.5, 155.0)
- added TP7: TestPoint_Small, TestPoint:TestPoint_Pad_D1.0mm, F.Cu at (250.5, 139.7)
- added TP8: TestPoint_Small, TestPoint:TestPoint_Pad_D1.0mm, F.Cu at (250.5, 124.4)
- added U23: PCA9306DC, Package_SO:VSSOP-8_2.3x2mm_P0.5mm, B.Cu at (20.0, 136.5)
- added U24: TXS0104EPW, Package_SO:TSSOP-14_4.4x5mm_P0.65mm, B.Cu at (20.0, 131.8)
- added U25: PCA9306DC, Package_SO:VSSOP-8_2.3x2mm_P0.5mm, B.Cu at (20.4, 160.8)
- added U28: TXS0104EPW, Package_SO:TSSOP-14_4.4x5mm_P0.65mm, B.Cu at (19.0, 155.6)
- C10, C12, C129, C130, C131, C15, C18, C19, C191, C192, C195, C196, C197, C198, C199, C20, C200, C201, C202, C203, C204, C205, C206, C207, C209, C21, C210, C211, C212, C213, C214, C215, C216, C22, C221, C222, C223, C224, C225, C226, C227, C228, C229, C23, C230, C231, C233, C234, C235, C236, C237, C24, C26, C27, C28, C33, C34, C35, C36, C38, C39, C40, C45, C46, C47, C48, C5, C50, C51, C52, C7, FB1, FB2, Q1, Q2, Q3, R109, R11, R110, R12, R15, R16, R17, R2, R23, R27, R28, R29, R30, R31, R33, R5, R6, R7, R71, R72, R73, R74, R75, R76, R77, R78, R79, R8, R80, R81, R82, R83, R84, R85, R86, R94, R95, U18, U19, U22, U3, U4, U5, U6, Y2: moved to B.Cu
- C232: value 100nF -> 22uF 25V; footprint Capacitor_SMD:C_0402_1005Metric -> Capacitor_SMD:C_1206_3216Metric; moved to B.Cu
- J3: footprint Connector_PCBEdge:BUS_PCIexpress_x16 -> CHIPSAlliance_Connector:PCIexpress_x16_FHFL
- J5: footprint Connector_Samtec:Samtec_FMC_ASP-134486-01_10x40_P1.27mm_Vertical -> CHIPSAlliance_Connector:Samtec_FMC_ASP-134486-01_10x40_P1.27mm_Vertical
- R100, R102: value 1k -> 240R 1%
- R103, R105: value 240R 1% -> 1k
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Connections:
- net /FMC HPC 0/FMC.CLK0_M2C+ renamed /FMC0.CLK0_M2C+
- net /FMC HPC 0/FMC.CLK0_M2C- renamed /FMC0.CLK0_M2C-
- net /FMC HPC 0/FMC.CLK1_M2C+ renamed /FMC0.CLK1_M2C+
- net /FMC HPC 0/FMC.CLK1_M2C- renamed /FMC0.CLK1_M2C-
- net /FMC HPC 0/FMC.CLK2_BID+ renamed /FMC0.CLK2_BID+
- net /FMC HPC 0/FMC.CLK2_BID- renamed /FMC0.CLK2_BID-
- net /FMC HPC 0/FMC.CLK3_BID+ renamed /FMC0.CLK3_BID+
- net /FMC HPC 0/FMC.CLK3_BID- renamed /FMC0.CLK3_BID-
- net /FMC HPC 0/FMC.CLK_DIR renamed /FMC0.CLK_DIR
- net /FMC HPC 0/FMC.DP0_C2M+ renamed /FMC0.DP0_C2M+
- net /FMC HPC 0/FMC.DP0_C2M- renamed /FMC0.DP0_C2M-
- net /FMC HPC 0/FMC.DP0_M2C+ renamed /FMC0.DP0_M2C+
- net /FMC HPC 0/FMC.DP0_M2C- renamed /FMC0.DP0_M2C-
- net /FMC HPC 0/FMC.DP1_C2M+ renamed /FMC0.DP1_C2M+
- net /FMC HPC 0/FMC.DP1_C2M- renamed /FMC0.DP1_C2M-
- net /FMC HPC 0/FMC.DP1_M2C+ renamed /FMC0.DP1_M2C+
- net /FMC HPC 0/FMC.DP1_M2C- renamed /FMC0.DP1_M2C-
- net /FMC HPC 0/FMC.DP2_C2M+ renamed /FMC0.DP2_C2M+
- net /FMC HPC 0/FMC.DP2_C2M- renamed /FMC0.DP2_C2M-
- net /FMC HPC 0/FMC.DP2_M2C+ renamed /FMC0.DP2_M2C+
- net /FMC HPC 0/FMC.DP2_M2C- renamed /FMC0.DP2_M2C-
- net /FMC HPC 0/FMC.DP3_C2M+ renamed /FMC0.DP3_C2M+
- net /FMC HPC 0/FMC.DP3_C2M- renamed /FMC0.DP3_C2M-
- net /FMC HPC 0/FMC.DP3_M2C+ renamed /FMC0.DP3_M2C+
- net /FMC HPC 0/FMC.DP3_M2C- renamed /FMC0.DP3_M2C-
- net /FMC HPC 0/FMC.DP4_C2M+ renamed /FMC0.DP4_C2M+
- net /FMC HPC 0/FMC.DP4_C2M- renamed /FMC0.DP4_C2M-
- net /FMC HPC 0/FMC.DP4_M2C+ renamed /FMC0.DP4_M2C+
- net /FMC HPC 0/FMC.DP4_M2C- renamed /FMC0.DP4_M2C-
- net /FMC HPC 0/FMC.DP5_C2M+ renamed /FMC0.DP5_C2M+
- net /FMC HPC 0/FMC.DP5_C2M- renamed /FMC0.DP5_C2M-
- net /FMC HPC 0/FMC.DP5_M2C+ renamed /FMC0.DP5_M2C+
- net /FMC HPC 0/FMC.DP5_M2C- renamed /FMC0.DP5_M2C-
- net /FMC HPC 0/FMC.DP6_C2M+ renamed /FMC0.DP6_C2M+
- net /FMC HPC 0/FMC.DP6_C2M- renamed /FMC0.DP6_C2M-
- net /FMC HPC 0/FMC.DP6_M2C+ renamed /FMC0.DP6_M2C+
- net /FMC HPC 0/FMC.DP6_M2C- renamed /FMC0.DP6_M2C-
- net /FMC HPC 0/FMC.DP7_C2M+ renamed /FMC0.DP7_C2M+
- net /FMC HPC 0/FMC.DP7_C2M- renamed /FMC0.DP7_C2M-
- net /FMC HPC 0/FMC.DP7_M2C+ renamed /FMC0.DP7_M2C+
- net /FMC HPC 0/FMC.DP7_M2C- renamed /FMC0.DP7_M2C-
- net /FMC HPC 0/FMC.DP8_C2M+ renamed /FMC0.DP8_C2M+
- net /FMC HPC 0/FMC.DP8_C2M- renamed /FMC0.DP8_C2M-
- net /FMC HPC 0/FMC.DP8_M2C+ renamed /FMC0.DP8_M2C+
- net /FMC HPC 0/FMC.DP8_M2C- renamed /FMC0.DP8_M2C-
- net /FMC HPC 0/FMC.DP9_C2M+ renamed /FMC0.DP9_C2M+
- net /FMC HPC 0/FMC.DP9_C2M- renamed /FMC0.DP9_C2M-
- net /FMC HPC 0/FMC.DP9_M2C+ renamed /FMC0.DP9_M2C+
- net /FMC HPC 0/FMC.DP9_M2C- renamed /FMC0.DP9_M2C-
- net /FMC HPC 0/FMC.GBTCLK0+ renamed /FMC0.GBTCLK0+
- net /FMC HPC 0/FMC.GBTCLK0- renamed /FMC0.GBTCLK0-
- net /FMC HPC 0/FMC.GBTCLK1+ renamed /FMC0.GBTCLK1+
- net /FMC HPC 0/FMC.GBTCLK1- renamed /FMC0.GBTCLK1-
- net /FMC HPC 0/FMC.HA00_CC+ renamed /FMC0.HA00_CC+
- net /FMC HPC 0/FMC.HA00_CC- renamed /FMC0.HA00_CC-
- net /FMC HPC 0/FMC.HA01_CC+ renamed /FMC0.HA01_CC+
- net /FMC HPC 0/FMC.HA01_CC- renamed /FMC0.HA01_CC-
- net /FMC HPC 0/FMC.HA02+ renamed /FMC0.HA02+
- net /FMC HPC 0/FMC.HA02- renamed /FMC0.HA02-
- net /FMC HPC 0/FMC.HA03+ renamed /FMC0.HA03+
- net /FMC HPC 0/FMC.HA03- renamed /FMC0.HA03-
- net /FMC HPC 0/FMC.HA04+ renamed /FMC0.HA04+
- net /FMC HPC 0/FMC.HA04- renamed /FMC0.HA04-
- net /FMC HPC 0/FMC.HA05+ renamed /FMC0.HA05+
- net /FMC HPC 0/FMC.HA05- renamed /FMC0.HA05-
- net /FMC HPC 0/FMC.HA06+ renamed /FMC0.HA06+
- net /FMC HPC 0/FMC.HA06- renamed /FMC0.HA06-
- net /FMC HPC 0/FMC.HA07+ renamed /FMC0.HA07+
- net /FMC HPC 0/FMC.HA07- renamed /FMC0.HA07-
- net /FMC HPC 0/FMC.HA08+ renamed /FMC0.HA08+
- net /FMC HPC 0/FMC.HA08- renamed /FMC0.HA08-
- net /FMC HPC 0/FMC.HA09+ renamed /FMC0.HA09+
- net /FMC HPC 0/FMC.HA09- renamed /FMC0.HA09-
- net /FMC HPC 0/FMC.HA10+ renamed /FMC0.HA10+
- net /FMC HPC 0/FMC.HA10- renamed /FMC0.HA10-
- net /FMC HPC 0/FMC.HA11+ renamed /FMC0.HA11+
- net /FMC HPC 0/FMC.HA11- renamed /FMC0.HA11-
- net /FMC HPC 0/FMC.HA12+ renamed /FMC0.HA12+
- net /FMC HPC 0/FMC.HA12- renamed /FMC0.HA12-
- net /FMC HPC 0/FMC.HA13+ renamed /FMC0.HA13+
- net /FMC HPC 0/FMC.HA13- renamed /FMC0.HA13-
- net /FMC HPC 0/FMC.HA14+ renamed /FMC0.HA14+
- net /FMC HPC 0/FMC.HA14- renamed /FMC0.HA14-
- net /FMC HPC 0/FMC.HA15+ renamed /FMC0.HA15+
- net /FMC HPC 0/FMC.HA15- renamed /FMC0.HA15-
- net /FMC HPC 0/FMC.HA16+ renamed /FMC0.HA16+
- net /FMC HPC 0/FMC.HA16- renamed /FMC0.HA16-
- net /FMC HPC 0/FMC.HA17_CC+ renamed /FMC0.HA17_CC+
- net /FMC HPC 0/FMC.HA17_CC- renamed /FMC0.HA17_CC-
- net /FMC HPC 0/FMC.HA18+ renamed /FMC0.HA18+
- net /FMC HPC 0/FMC.HA18- renamed /FMC0.HA18-
- net /FMC HPC 0/FMC.HA19+ renamed /FMC0.HA19+
- net /FMC HPC 0/FMC.HA19- renamed /FMC0.HA19-
- net /FMC HPC 0/FMC.HA20+ renamed /FMC0.HA20+
- net /FMC HPC 0/FMC.HA20- renamed /FMC0.HA20-
- net /FMC HPC 0/FMC.HA21+ renamed /FMC0.HA21+
- net /FMC HPC 0/FMC.HA21- renamed /FMC0.HA21-
- net /FMC HPC 0/FMC.HA22+ renamed /FMC0.HA22+
- net /FMC HPC 0/FMC.HA22- renamed /FMC0.HA22-
- net /FMC HPC 0/FMC.HA23+ renamed /FMC0.HA23+
- net /FMC HPC 0/FMC.HA23- renamed /FMC0.HA23-
- net /FMC HPC 0/FMC.HB00_CC+ renamed /FMC0.HB00_CC+
- net /FMC HPC 0/FMC.HB00_CC- renamed /FMC0.HB00_CC-
- net /FMC HPC 0/FMC.HB01+ renamed /FMC0.HB01+
- net /FMC HPC 0/FMC.HB01- renamed /FMC0.HB01-
- net /FMC HPC 0/FMC.HB02+ renamed /FMC0.HB02+
- net /FMC HPC 0/FMC.HB02- renamed /FMC0.HB02-
- net /FMC HPC 0/FMC.HB03+ renamed /FMC0.HB03+
- net /FMC HPC 0/FMC.HB03- renamed /FMC0.HB03-
- net /FMC HPC 0/FMC.HB04+ renamed /FMC0.HB04+
- net /FMC HPC 0/FMC.HB04- renamed /FMC0.HB04-
- net /FMC HPC 0/FMC.HB05+ renamed /FMC0.HB05+
- net /FMC HPC 0/FMC.HB05- renamed /FMC0.HB05-
- net /FMC HPC 0/FMC.HB06_CC+ renamed /FMC0.HB06_CC+
- net /FMC HPC 0/FMC.HB06_CC- renamed /FMC0.HB06_CC-
- net /FMC HPC 0/FMC.HB07+ renamed /FMC0.HB07+
- net /FMC HPC 0/FMC.HB07- renamed /FMC0.HB07-
- net /FMC HPC 0/FMC.HB08+ renamed /FMC0.HB08+
- net /FMC HPC 0/FMC.HB08- renamed /FMC0.HB08-
- net /FMC HPC 0/FMC.HB09+ renamed /FMC0.HB09+
- net /FMC HPC 0/FMC.HB09- renamed /FMC0.HB09-
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Other:
- board size 84.3 x 8.4 mm -> 312 x 111.1 mm
- copper layers 8 -> 12
