File: fpga_candelabra/power_monitor.kicad_sch (KiCad schematic)
At the start: 20 parts, among them SW2 TS-1187A, U34 TPS386000

Commit message: fpga_candelabra: first rev fixes - fix vccint power stage FCCM mode - add ddr4 vref decoupling cap - refactor status LEDs - minor layout changes
Signed-off-by: Yichuan Gao <gaoyichuan000@gmail.com>
Parts:
- R182: value 0R -> DNP/0R; now not fitted
- SW2: value TS-1187A -> KMR223GLFG; footprint Button_Switch_SMD:SW_Push_1P1T_XKB_TS-1187A -> Button_Switch_SMD:SW_Push_1P1T_NO_CK_KMR2; LCSC Part C318884 -> C221678
Changed lines of the file:
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@@
 		(in_bom yes)
 		(on_board yes)
-		(dnp no)
+		(dnp yes)
 		(fields_autoplaced yes)
 		(property "Reference" "R182"
@@
 			)
 		)
-		(property "Value" "0R"
+		(property "Value" "DNP/0R"
 			(at 140.97 79.811 90)
 			(effects
@@
 				(path "/01ed9e92-4e50-4b41-90dc-10444aaec5f7/5dc37b92-8b79-4447-bbff-3e1051343fd5"
 					(reference "R182")
+					(unit 1)
+				)
+			)
+		)
+	)
+	(symbol
+		(lib_id "Switch:SW_Push")
+		(at 95.25 86.36 90)
+		(unit 1)
+		(exclude_from_sim no)
+		(in_bom yes)
+		(on_board yes)
+		(dnp no)
+		(fields_autoplaced yes)
+		(property "Reference" "SW2"
+			(at 91.5671 85.1478 90)
+			(effects
+				(font
+					(size 1.27 1.27)
+				)
+				(justify left)
+			)
+		)
+		(property "Value" "KMR223GLFG"
+			(at 91.5671 87.5721 90)
+			(effects
+				(font
+					(size 1.27 1.27)
+				)
+				(justify left)
+			)
+		)
+		(property "Footprint" "Button_Switch_SMD:SW_Push_1P1T_NO_CK_KMR2"
+			(at 90.17 86.36 0)
+			(effects
+				(font
+					(size 1.27 1.27)
+				)
+				(hide yes)
+			)
+		)
+		(property "Datasheet" "~"
+			(at 90.17 86.36 0)
+			(effects
+				(font
+					(size 1.27 1.27)
+				)
+				(hide yes)
+			)
+		)
+		(property "Description" "Push button switch, generic, two pins"
+			(at 95.25 86.36 0)
+			(effects
+				(font
+					(size 1.27 1.27)
+				)
+				(hide yes)
+			)
+		)
+		(property "LCSC Part" "C221678"
+			(at 95.25 86.36 90)
+			(effects
+				(font
+					(size 1.27 1.27)
+				)
+				(hide yes)
+			)
+		)
+		(pin "1"
+		)
+		(pin "2"
+		)
+		(instances
+			(project "fpga_candelabra"
+				(path "/01ed9e92-4e50-4b41-90dc-10444aaec5f7/5dc37b92-8b79-4447-bbff-3e1051343fd5"
+					(reference "SW2")
 					(unit 1)
 				)
@@
 					(unit 1)
 				)
-			)
-		)
-	)
-	(symbol
-		(lib_id "Switch:SW_Push")
-		(at 95.25 86.36 90)
-		(unit 1)
-		(exclude_from_sim no)
-		(in_bom yes)
-		(on_board yes)
-		(dnp no)
-		(fields_autoplaced yes)
-		(property "Reference" "SW2"
-			(at 91.5671 85.1478 90)
-			(effects
-				(font
-					(size 1.27 1.27)
-				)
-				(justify left)
-			)
-		)
-		(property "Value" "TS-1187A"
-			(at 91.5671 87.5721 90)
-			(effects
-				(font
-					(size 1.27 1.27)
-				)
-				(justify left)
-			)
-		)
-		(property "Footprint" "Button_Switch_SMD:SW_Push_1P1T_XKB_TS-1187A"
-			(at 90.17 86.36 0)
-			(effects
-				(font
-					(size 1.27 1.27)
-				)
-				(hide yes)
-			)
-		)
-		(property "Datasheet" "~"
-			(at 90.17 86.36 0)
-			(effects
-				(font
-					(size 1.27 1.27)
-				)
-				(hide yes)
-			)
-		)
-		(property "Description" "Push button switch, generic, two pins"
-			(at 95.25 86.36 0)
-			(effects
-				(font
-					(size 1.27 1.27)
-				)
-				(hide yes)
-			)
-		)
-		(property "LCSC Part" "C318884"
-			(at 95.25 86.36 90)
-			(effects
-				(font
-					(size 1.27 1.27)
-				)
-				(hide yes)
-			)
-		)
-		(pin "1"
-		)
-		(pin "2"
-		)
-		(instances
-			(project "fpga_candelabra"
-				(path "/01ed9e92-4e50-4b41-90dc-10444aaec5f7/5dc37b92-8b79-4447-bbff-3e1051343fd5"
-					(reference "SW2")
-					(unit 1)
-				)

Commit message: fpga_candelabra: add author & rev to schematics
Signed-off-by: Yichuan Gao <gaoyichuan000@gmail.com>
Other:
- company: (none) -> CHIPS Alliance
- title: (none) -> Power Monitor Reset
Changed lines of the file:
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@@
 	(generator_version "8.0")
 	(paper "A4")
+	(title_block
+		(title "Power Monitor Reset")
+		(date "2025-02-05")
+		(rev "0.2.0")
+		(company "CHIPS Alliance")
+		(comment 1 "Yichuan Gao")
+		(comment 2 "Yichuan Gao")
+	)
 	(junction
 		(at 57.15 67.31)

Commit message: fpga_candelabra: update to kicad 9.0
Other:
- company: CHIPS Alliance -> Sipeed
