File: fpga_candelabra/power_monitor.kicad_sch (KiCad schematic)
At the start: 20 parts, among them SW2 KMR223GLFG, U34 TPS386000

Commit message: fpga_candelabra: update library and preserve schematic connections
Signed-off-by: Huang Rui <vowstar@gmail.com>
Other:
- moved on the sheet: U34
Changed lines of the file:
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@@
 	(wire
 		(pts
-			(xy 123.19 86.36) (xy 123.19 87.63)
-		)
-		(stroke
-			(width 0)
-			(type default)
-		)
-	)
-	(wire
-		(pts
-			(xy 123.19 34.29) (xy 123.19 35.56)
+			(xy 123.19 87.63) (xy 123.19 87.63)
+		)
+		(stroke
+			(width 0)
+			(type default)
+		)
+	)
+	(wire
+		(pts
+			(xy 123.19 34.29) (xy 123.19 36.83)
 		)
 		(stroke
@@
 	(wire
 		(pts
-			(xy 125.73 86.36) (xy 125.73 87.63)
+			(xy 125.73 87.63) (xy 125.73 87.63)
 		)
 		(stroke
@@
 	(symbol
 		(lib_id "CHIPSAlliance_Power_Supervisor:TPS386000")
-		(at 123.19 60.96 0)
+		(at 123.19 62.23 0)
 		(unit 1)
 		(body_style 1)
