File: fpga_candelabra/fpga_io_slr0.kicad_sch (KiCad schematic)
At the start: 1 part, among them U1 XCVU13P-B2104

Commit message: fpga_candelabra: update library and preserve schematic connections
Signed-off-by: Huang Rui <vowstar@gmail.com>
Parts:
- U1: footprint CHIPSAlliance_Package_BGA:Xilinx_FHGB2104_VU13P_PkgLength -> CHIPSAlliance_Package_BGA:Xilinx_FHGB2104_BGA-2104_52.5x52.5mm_Layout46x46_P1mm_Ball0.6mm_Pad0.5mm_NSMD_VU13P_PkgLength
Changed lines of the file:
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@@
 	(symbol
 		(lib_id "CHIPSAlliance_FPGA_Xilinx_Virtex_UltraScale_Plus:XCVU13P-B2104")
-		(at 172.72 24.13 0)
+		(at 195.58 90.17 0)
 		(unit 4)
 		(body_style 1)
@@
 			)
 		)
-		(property "Footprint" "CHIPSAlliance_Package_BGA:Xilinx_FHGB2104_VU13P_PkgLength"
+		(property "Footprint" "CHIPSAlliance_Package_BGA:Xilinx_FHGB2104_BGA-2104_52.5x52.5mm_Layout46x46_P1mm_Ball0.6mm_Pad0.5mm_NSMD_VU13P_PkgLength"
 			(at 171.45 22.86 0)
 			(hide yes)
@@
 	(symbol
 		(lib_id "CHIPSAlliance_FPGA_Xilinx_Virtex_UltraScale_Plus:XCVU13P-B2104")
-		(at 102.87 24.13 0)
+		(at 125.73 90.17 0)
 		(unit 3)
 		(body_style 1)
@@
 			)
 		)
-		(property "Footprint" "CHIPSAlliance_Package_BGA:Xilinx_FHGB2104_VU13P_PkgLength"
+		(property "Footprint" "CHIPSAlliance_Package_BGA:Xilinx_FHGB2104_BGA-2104_52.5x52.5mm_Layout46x46_P1mm_Ball0.6mm_Pad0.5mm_NSMD_VU13P_PkgLength"
 			(at 101.6 22.86 0)
 			(hide yes)
@@
 	(symbol
 		(lib_id "CHIPSAlliance_FPGA_Xilinx_Virtex_UltraScale_Plus:XCVU13P-B2104")
-		(at 30.48 24.13 0)
+		(at 53.34 90.17 0)
 		(unit 2)
 		(body_style 1)
@@
 			)
 		)
-		(property "Footprint" "CHIPSAlliance_Package_BGA:Xilinx_FHGB2104_VU13P_PkgLength"
+		(property "Footprint" "CHIPSAlliance_Package_BGA:Xilinx_FHGB2104_BGA-2104_52.5x52.5mm_Layout46x46_P1mm_Ball0.6mm_Pad0.5mm_NSMD_VU13P_PkgLength"
 			(at 29.21 22.86 0)
 			(hide yes)
