File: fpga_candelabra/fpga_io_slr1.kicad_sch (KiCad schematic)
At the start: 10 parts, among them U1 XCVU13P-B2104

Commit message: fpga_candelabra: update library and preserve schematic connections
Signed-off-by: Huang Rui <vowstar@gmail.com>
Parts:
- U1: footprint CHIPSAlliance_Package_BGA:Xilinx_FHGB2104_VU13P_PkgLength -> CHIPSAlliance_Package_BGA:Xilinx_FHGB2104_BGA-2104_52.5x52.5mm_Layout46x46_P1mm_Ball0.6mm_Pad0.5mm_NSMD_VU13P_PkgLength
Changed lines of the file:
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@@
 	(symbol
 		(lib_id "CHIPSAlliance_FPGA_Xilinx_Virtex_UltraScale_Plus:XCVU13P-B2104")
-		(at 238.76 25.4 0)
+		(at 261.62 91.44 0)
 		(unit 8)
 		(body_style 1)
@@
 			)
 		)
-		(property "Footprint" "CHIPSAlliance_Package_BGA:Xilinx_FHGB2104_VU13P_PkgLength"
+		(property "Footprint" "CHIPSAlliance_Package_BGA:Xilinx_FHGB2104_BGA-2104_52.5x52.5mm_Layout46x46_P1mm_Ball0.6mm_Pad0.5mm_NSMD_VU13P_PkgLength"
 			(at 237.49 24.13 0)
 			(hide yes)
@@
 	(symbol
 		(lib_id "CHIPSAlliance_FPGA_Xilinx_Virtex_UltraScale_Plus:XCVU13P-B2104")
-		(at 34.29 25.4 0)
+		(at 57.15 91.44 0)
 		(unit 5)
 		(body_style 1)
@@
 			)
 		)
-		(property "Footprint" "CHIPSAlliance_Package_BGA:Xilinx_FHGB2104_VU13P_PkgLength"
+		(property "Footprint" "CHIPSAlliance_Package_BGA:Xilinx_FHGB2104_BGA-2104_52.5x52.5mm_Layout46x46_P1mm_Ball0.6mm_Pad0.5mm_NSMD_VU13P_PkgLength"
 			(at 33.02 24.13 0)
 			(hide yes)
@@
 	(symbol
 		(lib_id "CHIPSAlliance_FPGA_Xilinx_Virtex_UltraScale_Plus:XCVU13P-B2104")
-		(at 158.75 25.4 0)
+		(at 181.61 91.44 0)
 		(unit 7)
 		(body_style 1)
@@
 			)
 		)
-		(property "Footprint" "CHIPSAlliance_Package_BGA:Xilinx_FHGB2104_VU13P_PkgLength"
+		(property "Footprint" "CHIPSAlliance_Package_BGA:Xilinx_FHGB2104_BGA-2104_52.5x52.5mm_Layout46x46_P1mm_Ball0.6mm_Pad0.5mm_NSMD_VU13P_PkgLength"
 			(at 157.48 24.13 0)
 			(hide yes)
