File: fpga_candelabra/fpga_mgt_slr1.kicad_sch (KiCad schematic)
At the start: 1 part, among them U1 XCVU13P-B2104

Commit message: fpga_candelabra: update library and preserve schematic connections
Signed-off-by: Huang Rui <vowstar@gmail.com>
Parts:
- U1: footprint CHIPSAlliance_Package_BGA:Xilinx_FHGB2104_VU13P_PkgLength -> CHIPSAlliance_Package_BGA:Xilinx_FHGB2104_BGA-2104_52.5x52.5mm_Layout46x46_P1mm_Ball0.6mm_Pad0.5mm_NSMD_VU13P_PkgLength
Changed lines of the file:
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@@
 	(symbol
 		(lib_id "CHIPSAlliance_FPGA_Xilinx_Virtex_UltraScale_Plus:XCVU13P-B2104")
-		(at 95.25 100.33 0)
+		(at 110.49 123.19 0)
 		(unit 26)
 		(body_style 1)
@@
 			)
 		)
-		(property "Footprint" "CHIPSAlliance_Package_BGA:Xilinx_FHGB2104_VU13P_PkgLength"
+		(property "Footprint" "CHIPSAlliance_Package_BGA:Xilinx_FHGB2104_BGA-2104_52.5x52.5mm_Layout46x46_P1mm_Ball0.6mm_Pad0.5mm_NSMD_VU13P_PkgLength"
 			(at 93.98 99.06 0)
 			(hide yes)
@@
 	(symbol
 		(lib_id "CHIPSAlliance_FPGA_Xilinx_Virtex_UltraScale_Plus:XCVU13P-B2104")
-		(at 209.55 100.33 0)
+		(at 224.79 123.19 0)
 		(unit 28)
 		(body_style 1)
@@
 			)
 		)
-		(property "Footprint" "CHIPSAlliance_Package_BGA:Xilinx_FHGB2104_VU13P_PkgLength"
+		(property "Footprint" "CHIPSAlliance_Package_BGA:Xilinx_FHGB2104_BGA-2104_52.5x52.5mm_Layout46x46_P1mm_Ball0.6mm_Pad0.5mm_NSMD_VU13P_PkgLength"
 			(at 208.28 99.06 0)
 			(hide yes)
@@
 	(symbol
 		(lib_id "CHIPSAlliance_FPGA_Xilinx_Virtex_UltraScale_Plus:XCVU13P-B2104")
-		(at 33.02 31.75 0)
+		(at 48.26 54.61 0)
 		(unit 16)
 		(body_style 1)
@@
 			)
 		)
-		(property "Footprint" "CHIPSAlliance_Package_BGA:Xilinx_FHGB2104_VU13P_PkgLength"
+		(property "Footprint" "CHIPSAlliance_Package_BGA:Xilinx_FHGB2104_BGA-2104_52.5x52.5mm_Layout46x46_P1mm_Ball0.6mm_Pad0.5mm_NSMD_VU13P_PkgLength"
 			(at 31.75 30.48 0)
 			(hide yes)
@@
 	(symbol
 		(lib_id "CHIPSAlliance_FPGA_Xilinx_Virtex_UltraScale_Plus:XCVU13P-B2104")
-		(at 209.55 31.75 0)
+		(at 224.79 54.61 0)
 		(unit 19)
 		(body_style 1)
@@
 			)
 		)
-		(property "Footprint" "CHIPSAlliance_Package_BGA:Xilinx_FHGB2104_VU13P_PkgLength"
+		(property "Footprint" "CHIPSAlliance_Package_BGA:Xilinx_FHGB2104_BGA-2104_52.5x52.5mm_Layout46x46_P1mm_Ball0.6mm_Pad0.5mm_NSMD_VU13P_PkgLength"
 			(at 208.28 30.48 0)
 			(hide yes)
@@
 	(symbol
 		(lib_id "CHIPSAlliance_FPGA_Xilinx_Virtex_UltraScale_Plus:XCVU13P-B2104")
-		(at 95.25 31.75 0)
+		(at 110.49 54.61 0)
 		(unit 17)
 		(body_style 1)
@@
 			)
 		)
-		(property "Footprint" "CHIPSAlliance_Package_BGA:Xilinx_FHGB2104_VU13P_PkgLength"
+		(property "Footprint" "CHIPSAlliance_Package_BGA:Xilinx_FHGB2104_BGA-2104_52.5x52.5mm_Layout46x46_P1mm_Ball0.6mm_Pad0.5mm_NSMD_VU13P_PkgLength"
 			(at 93.98 30.48 0)
 			(hide yes)
@@
 	(symbol
 		(lib_id "CHIPSAlliance_FPGA_Xilinx_Virtex_UltraScale_Plus:XCVU13P-B2104")
-		(at 152.4 31.75 0)
+		(at 167.64 54.61 0)
 		(unit 18)
 		(body_style 1)
@@
 			)
 		)
-		(property "Footprint" "CHIPSAlliance_Package_BGA:Xilinx_FHGB2104_VU13P_PkgLength"
+		(property "Footprint" "CHIPSAlliance_Package_BGA:Xilinx_FHGB2104_BGA-2104_52.5x52.5mm_Layout46x46_P1mm_Ball0.6mm_Pad0.5mm_NSMD_VU13P_PkgLength"
 			(at 151.13 30.48 0)
 			(hide yes)
@@
 	(symbol
 		(lib_id "CHIPSAlliance_FPGA_Xilinx_Virtex_UltraScale_Plus:XCVU13P-B2104")
-		(at 152.4 100.33 0)
+		(at 167.64 123.19 0)
 		(unit 27)
 		(body_style 1)
@@
 			)
 		)
-		(property "Footprint" "CHIPSAlliance_Package_BGA:Xilinx_FHGB2104_VU13P_PkgLength"
+		(property "Footprint" "CHIPSAlliance_Package_BGA:Xilinx_FHGB2104_BGA-2104_52.5x52.5mm_Layout46x46_P1mm_Ball0.6mm_Pad0.5mm_NSMD_VU13P_PkgLength"
 			(at 151.13 99.06 0)
 			(hide yes)
@@
 	(symbol
 		(lib_id "CHIPSAlliance_FPGA_Xilinx_Virtex_UltraScale_Plus:XCVU13P-B2104")
-		(at 33.02 100.33 0)
+		(at 48.26 123.19 0)
 		(unit 25)
 		(body_style 1)
@@
 			)
 		)
-		(property "Footprint" "CHIPSAlliance_Package_BGA:Xilinx_FHGB2104_VU13P_PkgLength"
+		(property "Footprint" "CHIPSAlliance_Package_BGA:Xilinx_FHGB2104_BGA-2104_52.5x52.5mm_Layout46x46_P1mm_Ball0.6mm_Pad0.5mm_NSMD_VU13P_PkgLength"
 			(at 31.75 99.06 0)
 			(hide yes)
