File: fpga_candelabra/fpga_mgt_slr2.kicad_sch (KiCad schematic)
At the start: 1 part, among them U1 XCVU13P-B2104

Commit message: fpga_candelabra: update library and preserve schematic connections
Signed-off-by: Huang Rui <vowstar@gmail.com>
Parts:
- U1: footprint CHIPSAlliance_Package_BGA:Xilinx_FHGB2104_VU13P_PkgLength -> CHIPSAlliance_Package_BGA:Xilinx_FHGB2104_BGA-2104_52.5x52.5mm_Layout46x46_P1mm_Ball0.6mm_Pad0.5mm_NSMD_VU13P_PkgLength
Changed lines of the file:
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@@
 	(symbol
 		(lib_id "CHIPSAlliance_FPGA_Xilinx_Virtex_UltraScale_Plus:XCVU13P-B2104")
-		(at 166.37 29.21 0)
+		(at 181.61 52.07 0)
 		(unit 22)
 		(body_style 1)
@@
 			)
 		)
-		(property "Footprint" "CHIPSAlliance_Package_BGA:Xilinx_FHGB2104_VU13P_PkgLength"
+		(property "Footprint" "CHIPSAlliance_Package_BGA:Xilinx_FHGB2104_BGA-2104_52.5x52.5mm_Layout46x46_P1mm_Ball0.6mm_Pad0.5mm_NSMD_VU13P_PkgLength"
 			(at 165.1 27.94 0)
 			(hide yes)
@@
 	(symbol
 		(lib_id "CHIPSAlliance_FPGA_Xilinx_Virtex_UltraScale_Plus:XCVU13P-B2104")
-		(at 223.52 29.21 0)
+		(at 238.76 52.07 0)
 		(unit 23)
 		(body_style 1)
@@
 			)
 		)
-		(property "Footprint" "CHIPSAlliance_Package_BGA:Xilinx_FHGB2104_VU13P_PkgLength"
+		(property "Footprint" "CHIPSAlliance_Package_BGA:Xilinx_FHGB2104_BGA-2104_52.5x52.5mm_Layout46x46_P1mm_Ball0.6mm_Pad0.5mm_NSMD_VU13P_PkgLength"
 			(at 222.25 27.94 0)
 			(hide yes)
@@
 	(symbol
 		(lib_id "CHIPSAlliance_FPGA_Xilinx_Virtex_UltraScale_Plus:XCVU13P-B2104")
-		(at 223.52 99.06 0)
+		(at 238.76 121.92 0)
 		(unit 32)
 		(body_style 1)
@@
 			)
 		)
-		(property "Footprint" "CHIPSAlliance_Package_BGA:Xilinx_FHGB2104_VU13P_PkgLength"
+		(property "Footprint" "CHIPSAlliance_Package_BGA:Xilinx_FHGB2104_BGA-2104_52.5x52.5mm_Layout46x46_P1mm_Ball0.6mm_Pad0.5mm_NSMD_VU13P_PkgLength"
 			(at 222.25 97.79 0)
 			(hide yes)
@@
 	(symbol
 		(lib_id "CHIPSAlliance_FPGA_Xilinx_Virtex_UltraScale_Plus:XCVU13P-B2104")
-		(at 109.22 99.06 0)
+		(at 124.46 121.92 0)
 		(unit 30)
 		(body_style 1)
@@
 			)
 		)
-		(property "Footprint" "CHIPSAlliance_Package_BGA:Xilinx_FHGB2104_VU13P_PkgLength"
+		(property "Footprint" "CHIPSAlliance_Package_BGA:Xilinx_FHGB2104_BGA-2104_52.5x52.5mm_Layout46x46_P1mm_Ball0.6mm_Pad0.5mm_NSMD_VU13P_PkgLength"
 			(at 107.95 97.79 0)
 			(hide yes)
@@
 	(symbol
 		(lib_id "CHIPSAlliance_FPGA_Xilinx_Virtex_UltraScale_Plus:XCVU13P-B2104")
-		(at 50.8 29.21 0)
+		(at 66.04 52.07 0)
 		(unit 20)
 		(body_style 1)
@@
 			)
 		)
-		(property "Footprint" "CHIPSAlliance_Package_BGA:Xilinx_FHGB2104_VU13P_PkgLength"
+		(property "Footprint" "CHIPSAlliance_Package_BGA:Xilinx_FHGB2104_BGA-2104_52.5x52.5mm_Layout46x46_P1mm_Ball0.6mm_Pad0.5mm_NSMD_VU13P_PkgLength"
 			(at 49.53 27.94 0)
 			(hide yes)
@@
 	(symbol
 		(lib_id "CHIPSAlliance_FPGA_Xilinx_Virtex_UltraScale_Plus:XCVU13P-B2104")
-		(at 109.22 29.21 0)
+		(at 124.46 52.07 0)
 		(unit 21)
 		(body_style 1)
@@
 			)
 		)
-		(property "Footprint" "CHIPSAlliance_Package_BGA:Xilinx_FHGB2104_VU13P_PkgLength"
+		(property "Footprint" "CHIPSAlliance_Package_BGA:Xilinx_FHGB2104_BGA-2104_52.5x52.5mm_Layout46x46_P1mm_Ball0.6mm_Pad0.5mm_NSMD_VU13P_PkgLength"
 			(at 107.95 27.94 0)
 			(hide yes)
@@
 	(symbol
 		(lib_id "CHIPSAlliance_FPGA_Xilinx_Virtex_UltraScale_Plus:XCVU13P-B2104")
-		(at 50.8 99.06 0)
+		(at 66.04 121.92 0)
 		(unit 29)
 		(body_style 1)
@@
 			)
 		)
-		(property "Footprint" "CHIPSAlliance_Package_BGA:Xilinx_FHGB2104_VU13P_PkgLength"
+		(property "Footprint" "CHIPSAlliance_Package_BGA:Xilinx_FHGB2104_BGA-2104_52.5x52.5mm_Layout46x46_P1mm_Ball0.6mm_Pad0.5mm_NSMD_VU13P_PkgLength"
 			(at 49.53 97.79 0)
 			(hide yes)
@@
 	(symbol
 		(lib_id "CHIPSAlliance_FPGA_Xilinx_Virtex_UltraScale_Plus:XCVU13P-B2104")
-		(at 166.37 99.06 0)
+		(at 181.61 121.92 0)
 		(unit 31)
 		(body_style 1)
@@
 			)
 		)
-		(property "Footprint" "CHIPSAlliance_Package_BGA:Xilinx_FHGB2104_VU13P_PkgLength"
+		(property "Footprint" "CHIPSAlliance_Package_BGA:Xilinx_FHGB2104_BGA-2104_52.5x52.5mm_Layout46x46_P1mm_Ball0.6mm_Pad0.5mm_NSMD_VU13P_PkgLength"
 			(at 165.1 97.79 0)
 			(hide yes)
