File: fpga_candelabra/fpga_power.kicad_sch (KiCad schematic)
At the start: 12 parts, among them U1 XCVU13P-B2104

Commit message: fpga_candelabra: update library and preserve schematic connections
Signed-off-by: Huang Rui <vowstar@gmail.com>
Parts:
- U1: footprint CHIPSAlliance_Package_BGA:Xilinx_FHGB2104_VU13P_PkgLength -> CHIPSAlliance_Package_BGA:Xilinx_FHGB2104_BGA-2104_52.5x52.5mm_Layout46x46_P1mm_Ball0.6mm_Pad0.5mm_NSMD_VU13P_PkgLength
Changed lines of the file:
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@@
 	(symbol
 		(lib_id "CHIPSAlliance_FPGA_Xilinx_Virtex_UltraScale_Plus:XCVU13P-B2104")
-		(at 44.45 49.53 0)
+		(at 57.15 72.39 0)
 		(unit 35)
 		(body_style 1)
@@
 			)
 		)
-		(property "Footprint" "CHIPSAlliance_Package_BGA:Xilinx_FHGB2104_VU13P_PkgLength"
+		(property "Footprint" "CHIPSAlliance_Package_BGA:Xilinx_FHGB2104_BGA-2104_52.5x52.5mm_Layout46x46_P1mm_Ball0.6mm_Pad0.5mm_NSMD_VU13P_PkgLength"
 			(at 43.18 48.26 0)
 			(hide yes)
@@
 	(symbol
 		(lib_id "CHIPSAlliance_FPGA_Xilinx_Virtex_UltraScale_Plus:XCVU13P-B2104")
-		(at 118.11 49.53 0)
+		(at 133.35 72.39 0)
 		(unit 36)
 		(body_style 1)
@@
 			)
 		)
-		(property "Footprint" "CHIPSAlliance_Package_BGA:Xilinx_FHGB2104_VU13P_PkgLength"
+		(property "Footprint" "CHIPSAlliance_Package_BGA:Xilinx_FHGB2104_BGA-2104_52.5x52.5mm_Layout46x46_P1mm_Ball0.6mm_Pad0.5mm_NSMD_VU13P_PkgLength"
 			(at 116.84 48.26 0)
 			(hide yes)
