File: fpga_candelabra/ipex_extension.kicad_sch (KiCad schematic)
At the start: 5 parts

Commit message: fpga_candelabra: update library and preserve schematic connections
Signed-off-by: Huang Rui <vowstar@gmail.com>
Parts:
- IPEX0, IPEX1, IPEX2, IPEX3: footprint CHIPSAlliance_Connector:I-PEX_20455-040E-76 -> CHIPSAlliance_Connector:I-PEX_20455-040E-76_1x40_P0.5mm_Horizontal
- IPEX4: footprint CHIPSAlliance_Connector:I-PEX_20455-050E-76 -> CHIPSAlliance_Connector:I-PEX_20455-050E-76_1x50_P0.5mm_Horizontal
Changed lines of the file:
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@@
 			)
 		)
-		(property "Footprint" "CHIPSAlliance_Connector:I-PEX_20455-040E-76"
+		(property "Footprint" "CHIPSAlliance_Connector:I-PEX_20455-040E-76_1x40_P0.5mm_Horizontal"
 			(at 88.9 71.12 0)
 			(effects
@@
 			)
 		)
-		(property "Footprint" "CHIPSAlliance_Connector:I-PEX_20455-050E-76"
+		(property "Footprint" "CHIPSAlliance_Connector:I-PEX_20455-050E-76_1x50_P0.5mm_Horizontal"
 			(at 260.35 83.82 0)
 			(effects
@@
 			)
 		)
-		(property "Footprint" "CHIPSAlliance_Connector:I-PEX_20455-040E-76"
+		(property "Footprint" "CHIPSAlliance_Connector:I-PEX_20455-040E-76_1x40_P0.5mm_Horizontal"
 			(at 165.1 71.12 0)
 			(effects
@@
 			)
 		)
-		(property "Footprint" "CHIPSAlliance_Connector:I-PEX_20455-040E-76"
+		(property "Footprint" "CHIPSAlliance_Connector:I-PEX_20455-040E-76_1x40_P0.5mm_Horizontal"
 			(at 127 71.12 0)
 			(effects
@@
 			)
 		)
-		(property "Footprint" "CHIPSAlliance_Connector:I-PEX_20455-040E-76"
+		(property "Footprint" "CHIPSAlliance_Connector:I-PEX_20455-040E-76_1x40_P0.5mm_Horizontal"
 			(at 50.8 71.12 0)
 			(effects
