File: fpga_candelabra/mikrobus.kicad_sch (KiCad schematic)
At the start: 19 parts, among them J6 Conn_mikroBUS_Host_2x8, U23 LSF0108PW, U24 LSF0108PW

Commit message: fpga_candelabra: update library and preserve schematic connections
Signed-off-by: Huang Rui <vowstar@gmail.com>
Parts:
- J6: footprint CHIPSAlliance_Connector:Conn_mikroBUS_Host_2x8_P2.54mm -> CHIPSAlliance_Connector:Conn_mikroBUS_Host_2x08_P2.54mm
Changed lines of the file:
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@@
 	(symbol
 		(lib_id "CHIPSAlliance_Connector:Conn_mikroBUS_Host_2x8")
-		(at 209.55 53.34 0)
+		(at 208.28 53.34 0)
 		(unit 1)
 		(body_style 1)
@@
 			)
 		)
-		(property "Footprint" "CHIPSAlliance_Connector:Conn_mikroBUS_Host_2x8_P2.54mm"
+		(property "Footprint" "CHIPSAlliance_Connector:Conn_mikroBUS_Host_2x08_P2.54mm"
 			(at 198.755 53.975 0)
 			(hide yes)
