File: fpga_candelabra/qsfp_conn.kicad_sch (KiCad schematic)
At the start: 28 parts, among them J7 QSFP+, U30 LSF0108PW

Commit message: fpga_candelabra: update library and preserve schematic connections
Signed-off-by: Huang Rui <vowstar@gmail.com>
Changed lines of the file:
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@@
 	(symbol
 		(lib_id "CHIPSAlliance_Interface:QSFP+")
-		(at 88.9 59.69 0)
+		(at 88.9 62.23 0)
 		(unit 1)
 		(body_style 1)
