File: fmc_sdram/fmc_sdram.kicad_pcb (KiCad board)
At the start: 4 copper layers, 76.5 x 69 mm, 73 parts, among them J1 SAMTEC_ASP-134604-01, J2 TYPE-C-31-M-12, J5 Conn_JTAG_20, SW7 TL3342F160QG, U1 M24C02-FMN, U10 SN74AVCH16T245GR, U11 SN74AVCH16T245GR, U12 SN74AVCH16T245GR, U13 SN74AVCH2T45DCU, U14 SN74AVCH2T45DCU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

Commit message: fmc_sdram: tie dqm level shifter dir pins to vadj and fix pcb
Signed-off-by: Huang Rui <vowstar@gmail.com>
Connections:
- U13 pad 5: /FMC/SDRAM_DQ_DIR -> VADJ
- U14 pad 5: /FMC/SDRAM_DQ_DIR -> VADJ
Routing:
- net /FMC/SDRAM_DQ_DIR: track 89.2 -> 80.0 mm, vias 5 -> 3
- net VADJ: track 41.8 -> 49.4 mm
- net /Level Shifter/HV.DQM0: track 9.89 -> 9.11 mm
