File: fmc_sdram/level_shifter.kicad_sch (KiCad schematic)
At the start: 32 parts, among them U10 SN74AVCH16T245GR, U11 SN74AVCH16T245GR, U12 SN74AVCH16T245GR, U13 SN74AVCH2T45DCU, U14 SN74AVCH2T45DCU, U9 SN74AVCH16T245GR

Commit message: fmc_sdram: fix package for SN74AVCH16T245GR
Signed-off-by: Yichuan Gao <gaoyichuan000@gmail.com>
Parts:
- U10, U11, U12, U9: footprint Package_SO:TSSOP-48_8x12.5mm_P0.5mm -> Package_SO:TSSOP-48_6.1x12.5mm_P0.5mm
Changed lines of the file:
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@@
 			)
 		)
-		(property "Footprint" "Package_SO:TSSOP-48_8x12.5mm_P0.5mm"
+		(property "Footprint" "Package_SO:TSSOP-48_6.1x12.5mm_P0.5mm"
 			(at 118.745 57.15 0)
 			(effects
@@
 			)
 		)
-		(property "Footprint" "Package_SO:TSSOP-48_8x12.5mm_P0.5mm"
+		(property "Footprint" "Package_SO:TSSOP-48_6.1x12.5mm_P0.5mm"
 			(at 241.935 57.15 0)
 			(effects
@@
 			)
 		)
-		(property "Footprint" "Package_SO:TSSOP-48_8x12.5mm_P0.5mm"
+		(property "Footprint" "Package_SO:TSSOP-48_6.1x12.5mm_P0.5mm"
 			(at 56.515 57.15 0)
 			(effects
@@
 			)
 		)
-		(property "Footprint" "Package_SO:TSSOP-48_8x12.5mm_P0.5mm"
+		(property "Footprint" "Package_SO:TSSOP-48_6.1x12.5mm_P0.5mm"
 			(at 183.515 57.15 0)
 			(effects

Commit message: fmc_sdram: tie dqm level shifter dir pins to vadj and fix pcb
Signed-off-by: Huang Rui <vowstar@gmail.com>
Connections:
- net SDRAM_DQ_DIR: no longer U13.5 (DIR), U14.5 (DIR)
- net VADJ: now also U13.5 (DIR), U14.5 (DIR)
